File: shinything/shinything.kicad_sch (KiCad schematic)
At the start: 63 parts, among them J1 Power In, SW1 SW_SPDT, U1 MT3608, U2 4017, U3 LM556

Commit message: Shiny thing lcsc parts and fixes
Parts:
- added H5: Centre Hole, MountingHole:MountingHole_2.5mm, symbol Mechanical:MountingHole
- added R19: 33k, Resistor_SMD:R_0805_2012Metric, symbol Device:R
- C1, C4: LCSC (none) -> C107179
- C2, C3, C7, C8: LCSC (none) -> C47971
- C5, C6: LCSC (none) -> C24497
- D1, D10, D11, D12, D13, D14, D15, D16, D17, D18, D19, D2, D20, D21, D22, D23, D24, D25, D26, D3, D4, D5, D6, D7, D8, D9: LCSC (none) -> C125099
- D30: LCSC (none) -> C232829
- L1: footprint Inductor_SMD:L_6.3x6.3_H3 -> Inductor_SMD:L_1210_3225Metric_Pad1.42x2.65mm_HandSolder; LCSC (none) -> C464437
- R1, R3: LCSC (none) -> C100047
- R10, R11, R12, R14, R15, R16, R17, R18, R5, R6, R7, R8, R9: LCSC (none) -> C105877
- R13, R4: LCSC (none) -> C137446
- R2: LCSC (none) -> C114526
- SW1: footprint Button_Switch_THT:SW_Slide_1P2T_CK_OS102011MS2Q -> Connector_PinSocket_2.54mm:PinSocket_1x03_P2.54mm_Vertical; LCSC (none) -> C92657
- U1: LCSC (none) -> C84817
- U2: LCSC (none) -> C11349
- U3: LCSC (none) -> C434479
Connections:
- net GND: now also U2.13 (CKEN)
- net VLOGIC: no longer U2.13 (CKEN)
- net at C7.1, U3.1 (DIS), U3.2 (THR): now also R19.2; no longer R13.2
- new net: R13.2, R19.1
Other:
- note added: "to get value 66k"
- note removed: "TODO: increase value >50k"
- moved on the sheet: R13

Commit message: Flashing lights thing
Parts:
- D1, D10, D11, D12, D13, D14, D15, D16, D17, D18, D19, D2, D20, D21, D22, D23, D24, D25, D26, D3, D4, D5, D6, D7, D8, D9: LCSC C125099 -> C125086
Connections:
- net VLOGIC: now also U3.10 (R), U3.4 (R)
- no-connect marks 3 -> 2
