File: shinything/shinything.kicad_pcb (KiCad board)
At the start: 2 copper layers, 52 x 52 mm, 63 parts, among them J1 Power In, SW1 SW_SPDT, U1 MT3608, U2 4017, U3 LM556

Commit message: Shiny thing lcsc parts and fixes
Parts:
- added H5: Centre Hole, MountingHole:MountingHole_2.5mm, F.Cu at (132.5, 93.5)
- added R19: 33k, Resistor_SMD:R_0805_2012Metric, F.Cu at (115.0, 96.5)
- L1: footprint Inductor_SMD:L_6.3x6.3_H3 -> Inductor_SMD:L_1210_3225Metric_Pad1.42x2.65mm_HandSolder
- R3: value 33k -> 10k
- R4: value 10k -> 33k
- SW1: footprint Button_Switch_THT:SW_Slide_1P2T_CK_OS102011MS2Q -> Connector_PinSocket_2.54mm:PinSocket_1x03_P2.54mm_Vertical
- moved D1 7.28 mm to (139.5, 92.5), turned to 0 degrees
- moved D2 7.28 mm to (139.5, 90.0), turned to 180 degrees
- moved R13 4.03 mm to (113.0, 99.5), turned to 90 degrees
- moved R5 1.50 mm to (135.0, 89.5), turned to 180 degrees
- turned SW1 to 180 degrees
Connections:
- R13 pad 2: Net-(C7-Pad1) -> Net-(R13-Pad2)
- U2 pad 13: VLOGIC -> GND
Routing:
- net VLOGIC: track 152.7 -> 138.5 mm, vias 17 -> 16
- net GND: track 49.7 -> 57.6 mm
- net /VBAT: track 9.35 -> 6.21 mm
- net Net-(R13-Pad2): track 0.00 -> 2.50 mm
- net /VBAT_SW: track 15.4 -> 16.6 mm
- net /COUNT0: track 39.6 -> 40.5 mm
- net Net-(D2-Pad2): track 3.22 -> 2.34 mm
- net Net-(C7-Pad1): track 5.77 -> 6.59 mm
- net Net-(D30-Pad2): track 9.40 -> 9.92 mm

Commit message: Flashing lights thing
Parts:
- moved R12 8.51 mm to (150.0, 89.0)
- moved D13 8.50 mm to (153.6, 82.0)
- moved D14 8.50 mm to (153.6, 79.5)
- moved D15 8.50 mm to (153.6, 90.5)
- moved D16 8.50 mm to (153.6, 88.0)
- moved R11 8.50 mm to (149.5, 80.5)
Connections:
- U3 pad 10: Net-(U3-Pad10) -> VLOGIC
- U3 pad 4: Net-(U3-Pad4) -> VLOGIC
Routing:
- net VLOGIC: track 138.5 -> 167.4 mm, vias 16 -> 18
- net /COUNT4: track 29.3 -> 21.2 mm
- net /COUNT3: track 24.3 -> 32.0 mm
- net Net-(C8-Pad1): track 13.7 -> 15.2 mm

Commit message: Maybe different pcb
Other:
- net class Default removed
Changed lines of the file:
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@@
-(kicad_pcb (version 20200518) (host pcbnew "5.99.0-unknown-60915fb~101~ubuntu18.04.1")
+(kicad_pcb (version 20200628) (host pcbnew "5.99.0-unknown-9f20c61~102~ubuntu18.04.1")
   (general
     (thickness 1.6)
@@
       (dielectric_constraints no)
     )
-    (last_trace_width 0.5)
-    (user_trace_width 0.5)
-    (user_trace_width 0.8)
-    (trace_clearance 0.2)
-    (zone_clearance 0.508)
-    (zone_45_only no)
-    (trace_min 0.2)
-    (clearance_min 0)
-    (via_min_annulus 0.05)
-    (via_min_size 0.4)
-    (through_hole_min 0.3)
-    (hole_to_hole_min 0.25)
-    (via_size 0.8)
-    (via_drill 0.4)
-    (uvia_size 0.3)
-    (uvia_drill 0.1)
-    (uvias_allowed no)
-    (uvia_min_size 0.2)
-    (uvia_min_drill 0.1)
-    (max_error 0.005)
-    (defaults
-      (edge_clearance 0.01)
-      (edge_cuts_line_width 0.05)
-      (courtyard_line_width 0.05)
-      (copper_line_width 0.2)
-      (copper_text_dims (size 1.5 1.5) (thickness 0.3))
-      (silk_line_width 0.12)
-      (silk_text_dims (size 1 1) (thickness 0.15))
-      (fab_layers_line_width 0.1)
-      (fab_layers_text_dims (size 1 1) (thickness 0.15))
-      (other_layers_line_width 0.1)
-      (other_layers_text_dims (size 1 1) (thickness 0.15))
-      (dimension_units 0)
-      (dimension_precision 1)
-    )
-    (pad_size 1.524 1.524)
-    (pad_drill 0.762)
-    (pad_to_mask_clearance 0.05)
     (aux_axis_origin 104.5 121)
     (grid_origin 104.5 121)
-    (visible_elements FFFDFF7F)
     (pcbplotparams
       (layerselection 0x010fc_ffffffff)
@@
       (outputformat 1)
       (mirror false)
-      (drillshape 1)
+      (drillshape 0)
       (scaleselection 1)
-      (outputdirectory "")
+      (outputdirectory "plot")
     )
   )
@@
   (net 52 "Net-(SW1-Pad3)")
   (net 53 "Net-(R13-Pad2)")
-  (net_class "Default" "This is the default net class."
-    (clearance 0.2)
-    (trace_width 0.25)
-    (via_dia 0.8)
-    (via_drill 0.4)
-    (uvia_dia 0.3)
-    (uvia_drill 0.1)
-    (add_net "/COUNT0")
-    (add_net "/COUNT1")
-    (add_net "/COUNT2")
-    (add_net "/COUNT3")
-    (add_net "/COUNT4")
-    (add_net "/COUNT5")
-    (add_net "/COUNT6")
-    (add_net "/COUNT7")
-    (add_net "/COUNT8")
-    (add_net "/COUNT9")
-    (add_net "/TIMER1")
-    (add_net "/TIMER2")
-    (add_net "/VBAT")
-    (add_net "/VBAT_SW")
-    (add_net "GND")
-    (add_net "Net-(C5-Pad1)")
-    (add_net "Net-(C6-Pad1)")
-    (add_net "Net-(C7-Pad1)")
-    (add_net "Net-(C8-Pad1)")
-    (add_net "Net-(D1-Pad2)")
-    (add_net "Net-(D10-Pad1)")
-    (add_net "Net-(D10-Pad2)")
-    (add_net "Net-(D11-Pad2)")
-    (add_net "Net-(D12-Pad2)")
-    (add_net "Net-(D13-Pad2)")
-    (add_net "Net-(D14-Pad2)")
-    (add_net "Net-(D15-Pad2)")
-    (add_net "Net-(D16-Pad2)")
-    (add_net "Net-(D17-Pad2)")
-    (add_net "Net-(D18-Pad2)")
-    (add_net "Net-(D19-Pad2)")
-    (add_net "Net-(D2-Pad2)")
-    (add_net "Net-(D20-Pad2)")
-    (add_net "Net-(D21-Pad2)")
-    (add_net "Net-(D22-Pad2)")
-    (add_net "Net-(D23-Pad2)")
-    (add_net "Net-(D24-Pad2)")
-    (add_net "Net-(D25-Pad2)")
-    (add_net "Net-(D26-Pad2)")
-    (add_net "Net-(D3-Pad2)")
-    (add_net "Net-(D30-Pad2)")
-    (add_net "Net-(D4-Pad2)")
-    (add_net "Net-(D5-Pad2)")
-    (add_net "Net-(D6-Pad2)")
-    (add_net "Net-(D7-Pad2)")
-    (add_net "Net-(D8-Pad2)")
-    (add_net "Net-(R1-Pad2)")
-    (add_net "Net-(R13-Pad2)")
-    (add_net "Net-(R3-Pad2)")
-    (add_net "Net-(SW1-Pad3)")
-    (add_net "Net-(U1-Pad6)")
-    (add_net "Net-(U2-Pad12)")
-    (add_net "VLOGIC")
-  )
   (module "Inductor_SMD:L_1210_3225Metric_Pad1.42x2.65mm_HandSolder" (layer "F.Cu")
     (at 118 82)
@@
     (fp_line (start -1.6 -1.25) (end 1.6 -1.25) (layer "F.Fab") (width 0.1))
     (fp_line (start -1.6 1.25) (end -1.6 -1.25) (layer "F.Fab") (width 0.1))
-    (pad "2" smd roundrect (at 1.4875 0) (size 1.425 2.65) (layers "F.Cu" "F.Paste" "F.Mask") (roundrect_rratio 0.175439)
+    (pad "2" smd roundrect (at 1.4875 0) (size 1.425 2.65) (layers "F.Cu" "F.Paste" "F.Mask") (roundrect_rratio 0.175439298245614)
       (net 46 "Net-(D30-Pad2)") (pinfunction "2"))
-    (pad "1" smd roundrect (at -1.4875 0) (size 1.425 2.65) (layers "F.Cu" "F.Paste" "F.Mask") (roundrect_rratio 0.175439)
+    (pad "1" smd roundrect (at -1.4875 0) (size 1.425 2.65) (layers "F.Cu" "F.Paste" "F.Mask") (roundrect_rratio 0.175439298245614)
       (net 3 "/VBAT_SW") (pinfunction "1"))
     (model "${KISYS3DMOD}/Inductor_SMD.3dshapes/L_1210_3225Metric.wrl"
@@
     (pad "2" thru_hole circle (at 5.4 0 90) (size 2.75 2.75) (drill 1.75) (layers *.Cu *.Mask)
       (net 47 "/VBAT") (pinfunction "Pin_2"))
-    (pad "1" thru_hole roundrect (at 0 0 90) (size 2.75 2.75) (drill 1.75) (layers *.Cu *.Mask) (roundrect_rratio 0.090909)
+    (pad "1" thru_hole roundrect (at 0 0 90) (size 2.75 2.75) (drill 1.75) (layers *.Cu *.Mask) (roundrect_rratio 0.09090909090909091)
       (net 1 "GND") (pinfunction "Pin_1"))
     (model "${KISYS3DMOD}/Connector_Wire.3dshapes/SolderWire-1sqmm_1x02_P5.4mm_D1.4mm_OD2.7mm.wrl"
