File: a7105-mr/a7105-mr.kicad_pcb (KiCad board)
At the start: 2 copper layers, 15.6 x 21.5 mm, 23 parts, among them J1 Conn_01x07_Male, J2 Conn_01x07_Male, U1 A7105, Y1 Crystal

Commit message: the reverse engineered module
Routing:
- net GND: track 8.43 -> 8.61 mm, vias 14 -> 22
Other:
- board size 15.6 x 21.5 mm -> 17.7 x 21.5 mm

Commit message: update bom
Parts:
- AE1: value Antenna_Chip -> SLDA52-2R540G-S1TF; footprint RF_Antenna:Texas_SWRA117D_2.4GHz_Left -> RF_Antenna:Johanson_2450AT43F0100
- J1, J2: footprint Connector_PinHeader_2.00mm:PinHeader_1x07_P2.00mm_Vertical -> a7105-mr:castellatedpads_7
- moved AE1 7.06 mm to (105.3, 106.5), turned to 180 degrees
- moved L4 3.95 mm to (108.2, 106.9), turned to 45 degrees
- moved C17 3.20 mm to (110.2, 106.4)
- moved L2 2.61 mm to (111.5, 108.0), turned to 0 degrees
Connections:
- AE1 pad 2: GND -> Net-(AE1-Pad2)
Routing:
- net GND: track 8.61 -> 7.41 mm, vias 22 -> 19
Other:
- board size 17.7 x 21.5 mm -> 15.6 x 16.8 mm

Commit message: A7105 module experiments
Parts:
- AE1: value SLDA52-2R540G-S1TF -> Antenna; footprint RF_Antenna:Johanson_2450AT43F0100 -> a7105-mr:MIFA2
- C14: value 27pF -> 22pF
- C15: value 33pF -> 22pF
- C3: value 10pF -> 22pF
- Y1: value Crystal -> X503216MSB2GI
- moved AE1 6.53 mm to (111.8, 105.5), turned to 0 degrees
- moved L4 3.32 mm to (111.5, 106.5), turned to -30 degrees
- moved C17 2.86 mm to (113.0, 107.0)
- moved L2 2.50 mm to (109.0, 108.0), turned to 90 degrees
Routing:
- net GND: vias 19 -> 18
Other:
- board size 15.6 x 16.8 mm -> 15.6 x 23 mm
- net class Default removed
