File: a7105-mr/a7105-mr.kicad_sch (KiCad schematic)
At the start: 23 parts, among them J1 Conn_01x07_Male, J2 Conn_01x07_Male, U1 A7105, Y1 X503216MSB2GI

Commit message: A7105 module experiments
Parts:
- removed AE1: SLDA52-2R540G-S1TF, RF_Antenna:Johanson_2450AT43F0100, symbol Device:Antenna_Chip
- added AE1: Antenna, a7105-mr:MIFA2, symbol Device:Antenna
- C1, C2, C4: LCSC C12530 -> C12530
- C5: LCSC C1525 -> C1525
Connections:
- net ANT: now also AE1.1 (A)
- no-connect marks 8 -> 7
Changed lines of the file:
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@@
   (junction (at 172.72 104.14) (diameter 0) (color 0 0 0 0))
   (no_connect (at 157.48 45.72))
-  (no_connect (at 96.52 45.72))
+  (no_connect (at 96.52 40.64))
+  (no_connect (at 157.48 53.34))
+  (no_connect (at 138.43 67.31))
   (no_connect (at 96.52 35.56))
   (no_connect (at 96.52 48.26))
-  (no_connect (at 96.52 40.64))
-  (no_connect (at 58.42 85.09))
-  (no_connect (at 138.43 67.31))
-  (no_connect (at 157.48 53.34))
+  (no_connect (at 96.52 45.72))
   (wire (pts (xy 58.42 90.17) (xy 67.31 90.17))
     (stroke (width 0) (type solid) (color 0 0 0 0))
@@
     )
   )
+  (symbol (lib_id "Device:Antenna") (at 58.42 85.09 0) (unit 1)
+    (in_bom yes) (on_board yes)
+    (property "Reference" "AE1" (id 0) (at 60.4521 85.3376 0)
+      (effects (font (size 1.27 1.27)) (justify left))
+    )
+    (property "Value" "Antenna" (id 1) (at 60.4521 87.6363 0)
+      (effects (font (size 1.27 1.27)) (justify left))
+    )
+    (property "Footprint" "a7105-mr:MIFA2" (id 2) (at 58.42 85.09 0)
+      (effects (font (size 1.27 1.27)) hide)
+    )
+    (property "Datasheet" "~" (id 3) (at 58.42 85.09 0)
+      (effects (font (size 1.27 1.27)) hide)
+    )
+  )
   (symbol (lib_id "Device:C") (at 67.31 93.98 0) (unit 1)
     (in_bom yes) (on_board yes)
@@
       (effects (font (size 1.27 1.27)) hide)
     )
-    (property "LCSC" " C12530" (id 4) (at 118.11 62.23 0)
+    (property "LCSC" "C12530" (id 4) (at 118.11 62.23 0)
       (effects (font (size 1.27 1.27)) hide)
     )
@@
       (effects (font (size 1.27 1.27)) hide)
     )
-    (property "LCSC" " C12530" (id 4) (at 130.81 52.07 0)
+    (property "LCSC" "C12530" (id 4) (at 130.81 52.07 0)
       (effects (font (size 1.27 1.27)) hide)
     )
@@
       (effects (font (size 1.27 1.27)) hide)
     )
-    (property "LCSC" " C1525" (id 4) (at 163.83 120.65 0)
+    (property "LCSC" "C1525" (id 4) (at 163.83 120.65 0)
       (effects (font (size 1.27 1.27)) hide)
     )
@@
       (effects (font (size 1.27 1.27)) hide)
     )
-    (property "LCSC" " C12530" (id 4) (at 165.1 90.17 0)
+    (property "LCSC" "C12530" (id 4) (at 165.1 90.17 0)
       (effects (font (size 1.27 1.27)) hide)
     )
@@
     )
   )
-  (symbol (lib_id "Device:Antenna_Chip") (at 55.88 87.63 90) (unit 1)
-    (in_bom yes) (on_board yes)
-    (property "Reference" "AE1" (id 0) (at 53.8226 79.6036 90))
-    (property "Value" "SLDA52-2R540G-S1TF " (id 1) (at 53.8226 81.915 90))
-    (property "Footprint" "RF_Antenna:Johanson_2450AT43F0100" (id 2) (at 51.435 90.17 0)
-      (effects (font (size 1.27 1.27)) hide)
-    )
-    (property "Datasheet" "~" (id 3) (at 51.435 90.17 0)
-      (effects (font (size 1.27 1.27)) hide)
-    )
-    (property "LCSC" "C279814" (id 4) (at 55.88 87.63 90)
-      (effects (font (size 1.27 1.27)) hide)
-    )
-  )
   (symbol (lib_id "Connector:Conn_01x07_Male") (at 91.44 43.18 0) (unit 1)
     (in_bom yes) (on_board yes)
@@
       (reference "#PWR0113") (unit 1)
     )
-    (path "/00000000-0000-0000-0000-00005e5b989c"
+    (path "/cf80728b-2b2d-4777-8b62-fbc5b743849d"
       (reference "AE1") (unit 1)
     )
