File: motorback/motorback.kicad_sch (KiCad schematic)
At the start: 9 parts, among them J1 Conn_01x03_Male, J2 Conn_01x01_Male, J3 Conn_01x01_Male, U1 DRV8837, U2 ATtiny412-SS

Commit message: motorback idea
Parts:
- removed U2: ATtiny412-SS, Package_SO:SOIC-8_3.9x4.9mm_P1.27mm, symbol MCU_Microchip_ATtiny:ATtiny412-SS
- added U2: ATtiny13V-10SSU, Package_SO:SOIC-8_3.9x4.9mm_P1.27mm, symbol MCU_Microchip_ATtiny:ATtiny13V-10SSU
- C2: value C -> 0.1uf
- D1: value 5v MM5Z5V1ST1G -> MM5Z5V1; LCSC (none) -> C55848
- J1: footprint Connector_PinHeader_2.00mm:PinHeader_1x03_P2.00mm_Vertical -> Connector_JST:JST_SH_SM03B-SRSS-TB_1x03-1MP_P1.00mm_Horizontal
Connections:
- net GND: now also U2.4 (GND)
- net MOTORF: now also U2.5 (PB0)
- net MOTORR: now also U2.6 (PB1)
- net PWMIN: now also U2.7 (PB2)
- net VLOGIC: now also U2.8 (VCC)
- no-connect marks 1 -> 3
