File: motorback_l/motorback_l.kicad_sch (KiCad schematic)
At the start: 10 parts, among them J1 Conn_01x03_Male, J2 Conn_01x01_Male, J3 Conn_01x01_Male, U1 DRV8837, U2 ATtiny13V-10SSU

Commit message: motorback update lcsc part numbers
Connections:
- net MOTORF: now also U1.5 (IN2); no longer U1.6 (IN1)
- net MOTORR: now also U1.6 (IN1); no longer U1.5 (IN2)
Other:
- note removed: "In-circuit programming pin mapping: PB5 (reset) - held low during programming PB0 - MOSI PB1 - MISO PB2 - SCK Program using a test-clip attached to the soic."
Changed lines of the file:
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@@
   (junction (at 182.88 63.5) (diameter 1.016) (color 0 0 0 0))
   (junction (at 200.66 63.5) (diameter 1.016) (color 0 0 0 0))
+  (no_connect (at 171.45 92.71))
   (no_connect (at 171.45 95.25))
-  (no_connect (at 171.45 92.71))
   (wire (pts (xy 36.83 43.18) (xy 66.04 43.18))
     (stroke (width 0) (type solid) (color 0 0 0 0))
@@
     (stroke (width 0) (type solid) (color 0 0 0 0))
   )
-  (wire (pts (xy 171.45 82.55) (xy 184.15 82.55))
+  (wire (pts (xy 171.45 82.55) (xy 201.93 82.55))
     (stroke (width 0) (type solid) (color 0 0 0 0))
   )
@@
     (stroke (width 0) (type solid) (color 0 0 0 0))
   )
-  (wire (pts (xy 184.15 81.28) (xy 207.01 81.28))
+  (wire (pts (xy 185.42 81.28) (xy 185.42 85.09))
     (stroke (width 0) (type solid) (color 0 0 0 0))
   )
-  (wire (pts (xy 184.15 82.55) (xy 184.15 81.28))
-    (stroke (width 0) (type solid) (color 0 0 0 0))
-  )
-  (wire (pts (xy 185.42 83.82) (xy 207.01 83.82))
-    (stroke (width 0) (type solid) (color 0 0 0 0))
-  )
-  (wire (pts (xy 185.42 85.09) (xy 185.42 83.82))
+  (wire (pts (xy 185.42 81.28) (xy 207.01 81.28))
     (stroke (width 0) (type solid) (color 0 0 0 0))
   )
@@
   )
   (wire (pts (xy 200.66 78.74) (xy 200.66 63.5))
+    (stroke (width 0) (type solid) (color 0 0 0 0))
+  )
+  (wire (pts (xy 201.93 82.55) (xy 201.93 83.82))
+    (stroke (width 0) (type solid) (color 0 0 0 0))
+  )
+  (wire (pts (xy 201.93 83.82) (xy 207.01 83.82))
     (stroke (width 0) (type solid) (color 0 0 0 0))
   )
@@
     (effects (font (size 1.27 1.27)) (justify right bottom))
   )
-  (text "In-circuit programming pin mapping:\n\nPB5 (reset) - held low during programming\nPB0 - MOSI\nPB1 - MISO\nPB2 - SCK\n\nProgram using a test-clip attached to the soic."
-    (at 93.98 119.38 0)
-    (effects (font (size 1.27 1.27)) (justify left bottom))
-  )
   (text "Zener diode regulates voltage\napprox 5v" (at 124.46 54.61 180)
