File: malenki-nanoi/malenki-nanoi.kicad_sch (KiCad schematic)
At the start: 14 parts, among them J1 Conn_01x02_Male-Connector, J2 Conn_01x08_Male, J3 Conn_01x02, U2 AIC1734-33GUTR, U3 ATtiny1616-M

Commit message: Assign manufacturer part numbers and lcsc numbers
Parts:
- C2, C3: LCSC (none) -> C19702; MPN (none) -> CL10A106KP8NNNC; Manufacturer (none) -> Samsung
- C4: LCSC (none) -> C1525; MPN (none) -> CL05B104KO5NNNC; Manufacturer (none) -> Samsung
- D1: MPN (none) -> 19-217/BHC-ZL1M2RY/3T; Manufacturer (none) -> Everlight
- D2: MPN (none) -> KT-0603R; Manufacturer (none) -> Hubei KENTO
- R1, R2: LCSC (none) -> C21190; MPN (none) -> 0603WAF1001T5E; Manufacturer (none) -> Uniroyal
- R3: LCSC (none) -> C4216; MPN (none) -> 0603WAF3302T5E; Manufacturer (none) -> Uniroyal
- R4: LCSC (none) -> C25804; MPN (none) -> 0603WAF1002T5E; Manufacturer (none) -> Uniroyal
- U2: MPN (none) -> AIC1734-33GUTR; Manufacturer (none) -> Analog Integrations
- U3: MPN (none) -> ATtiny1616-MNR; Manufacturer (none) -> MICROCHIP
Changed lines of the file:
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@@
   (junction (at 106.68 156.21) (diameter 1.016) (color 0 0 0 0))
   (junction (at 132.08 47.625) (diameter 1.016) (color 0 0 0 0))
+  (no_connect (at 127 52.705))
+  (no_connect (at 142.24 116.84))
   (no_connect (at 127 45.085))
-  (no_connect (at 142.24 116.84))
-  (no_connect (at 127 52.705))
+  (no_connect (at 127 57.785))
   (no_connect (at 111.76 114.3))
-  (no_connect (at 127 57.785))
   (wire (pts (xy 38.1 48.26) (xy 57.15 48.26))
     (stroke (width 0) (type solid) (color 0 0 0 0))
@@
       (effects (font (size 1.27 1.27)) hide)
     )
-    (property "LCSC" "" (id 5) (at 106.68 152.4 0)
+    (property "LCSC" "C4216" (id 5) (at 106.68 152.4 0)
+      (effects (font (size 1.27 1.27)) hide)
+    )
+    (property "MPN" "0603WAF3302T5E" (id 4) (at 106.68 152.4 0)
+      (effects (font (size 1.27 1.27)) hide)
+    )
+    (property "Manufacturer" "Uniroyal " (id 5) (at 106.68 152.4 0)
       (effects (font (size 1.27 1.27)) hide)
     )
@@
       (effects (font (size 1.27 1.27)) hide)
     )
-    (property "LCSC" "" (id 5) (at 106.68 160.02 0)
+    (property "LCSC" "C25804" (id 5) (at 106.68 160.02 0)
+      (effects (font (size 1.27 1.27)) hide)
+    )
+    (property "MPN" "0603WAF1002T5E" (id 4) (at 106.68 160.02 0)
+      (effects (font (size 1.27 1.27)) hide)
+    )
+    (property "Manufacturer" "Uniroyal" (id 5) (at 106.68 160.02 0)
       (effects (font (size 1.27 1.27)) hide)
     )
@@
       (effects (font (size 1.27 1.27)) hide)
     )
-    (property "LCSC" "" (id 5) (at 130.81 163.83 0)
+    (property "LCSC" "C21190" (id 5) (at 130.81 163.83 0)
+      (effects (font (size 1.27 1.27)) hide)
+    )
+    (property "MPN" "0603WAF1001T5E" (id 4) (at 130.81 163.83 0)
+      (effects (font (size 1.27 1.27)) hide)
+    )
+    (property "Manufacturer" "Uniroyal" (id 5) (at 130.81 163.83 0)
       (effects (font (size 1.27 1.27)) hide)
     )
@@
       (effects (font (size 1.27 1.27)) hide)
     )
-    (property "LCSC" "" (id 5) (at 146.05 163.83 0)
+    (property "LCSC" "C21190" (id 5) (at 146.05 163.83 0)
+      (effects (font (size 1.27 1.27)) hide)
+    )
+    (property "MPN" "0603WAF1001T5E" (id 4) (at 146.05 163.83 0)
+      (effects (font (size 1.27 1.27)) hide)
+    )
+    (property "Manufacturer" "Uniroyal" (id 5) (at 146.05 163.83 0)
       (effects (font (size 1.27 1.27)) hide)
     )
@@
       (effects (font (size 1.27 1.27)) hide)
     )
+    (property "MPN" "19-217/BHC-ZL1M2RY/3T" (id 4) (at 130.81 156.21 0)
+      (effects (font (size 1.27 1.27)) hide)
+    )
+    (property "Manufacturer" "Everlight" (id 5) (at 130.81 156.21 0)
+      (effects (font (size 1.27 1.27)) hide)
+    )
   )
   (symbol (lib_id "malenki-nano-rescue:LED-Device") (at 146.05 156.21 90) (unit 1)
@@
       (effects (font (size 1.27 1.27)) hide)
     )
+    (property "MPN" "KT-0603R" (id 4) (at 146.05 156.21 0)
+      (effects (font (size 1.27 1.27)) hide)
+    )
+    (property "Manufacturer" "Hubei KENTO" (id 5) (at 146.05 156.21 0)
+      (effects (font (size 1.27 1.27)) hide)
+    )
   )
   (symbol (lib_id "Connector_Generic:Conn_01x02") (at 173.99 49.53 0) (unit 1)
@@
       (effects (font (size 1.27 1.27)) hide)
     )
-    (property "LCSC" "" (id 5) (at 63.5 52.07 0)
+    (property "LCSC" "C19702" (id 5) (at 63.5 52.07 0)
+      (effects (font (size 1.27 1.27)) hide)
+    )
+    (property "MPN" "CL10A106KP8NNNC" (id 4) (at 63.5 52.07 0)
+      (effects (font (size 1.27 1.27)) hide)
+    )
+    (property "Manufacturer" "Samsung" (id 5) (at 63.5 52.07 0)
       (effects (font (size 1.27 1.27)) hide)
     )
@@
       (effects (font (size 1.27 1.27)) hide)
     )
-    (property "LCSC" "" (id 5) (at 92.71 52.07 0)
+    (property "LCSC" "C19702" (id 5) (at 92.71 52.07 0)
+      (effects (font (size 1.27 1.27)) hide)
+    )
+    (property "MPN" "CL10A106KP8NNNC" (id 4) (at 92.71 52.07 0)
+      (effects (font (size 1.27 1.27)) hide)
+    )
+    (property "Manufacturer" "Samsung" (id 5) (at 92.71 52.07 0)
       (effects (font (size 1.27 1.27)) hide)
     )
@@
       (effects (font (size 1.27 1.27)) hide)
     )
-    (property "LCSC" "" (id 5) (at 109.22 77.47 0)
+    (property "LCSC" "C1525" (id 5) (at 109.22 77.47 0)
+      (effects (font (size 1.27 1.27)) hide)
+    )
+    (property "MPN" "CL05B104KO5NNNC" (id 4) (at 109.22 77.47 0)
+      (effects (font (size 1.27 1.27)) hide)
+    )
+    (property "Manufacturer" "Samsung" (id 5) (at 109.22 77.47 0)
       (effects (font (size 1.27 1.27)) hide)
     )
@@
       (effects (font (size 1.27 1.27)) hide)
     )
+    (property "MPN" "AIC1734-33GUTR" (id 4) (at 80.01 44.45 0)
+      (effects (font (size 1.27 1.27)) hide)
+    )
+    (property "Manufacturer" "Analog Integrations" (id 5) (at 80.01 44.45 0)
+      (effects (font (size 1.27 1.27)) hide)
+    )
   )
   (symbol (lib_id "MCU_Microchip_ATtiny:ATtiny1616-M") (at 127 101.6 0) (unit 1)
@@
       (effects (font (size 1.27 1.27)) hide)
     )
+    (property "MPN" "ATtiny1616-MNR" (id 4) (at 127 101.6 0)
+      (effects (font (size 1.27 1.27)) hide)
+    )
+    (property "Manufacturer" "MICROCHIP" (id 5) (at 127 101.6 0)
+      (effects (font (size 1.27 1.27)) hide)
+    )
