File: beetleback_cg/beetleback_cg.kicad_sch (KiCad schematic)
At the start: 29 parts, among them J1 signalin, J2 powerin, J3 motor_pad_1, J4 motor_pad_2, Q1 IRF8313PBF, Q2 IRF8313PBF, U1 ATtiny13A-SS, U2 ADP3110A, U3 HT7550-2, U4 ADP3110A, U5 HT75C0-2

Commit message: Beetleback, Chipageddon edition
Parts:
- C1, C2, C3, C4, C8, C9: value 2.2uF 50V -> 1uF 25v; LCSC C50254 -> C52923
Changed lines of the file:
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@@
       (effects (font (size 1.27 1.27)) (justify left))
     )
-    (property "Value" "2.2uF 50V" (id 1) (at 62.6111 126.2443 0)
+    (property "Value" "1uF 25v" (id 1) (at 62.6111 126.2443 0)
       (effects (font (size 1.27 1.27)) (justify left))
     )
@@
       (effects (font (size 1.27 1.27)) hide)
     )
-    (property "LCSC" "C50254" (id 4) (at 59.69 125.095 0)
+    (property "LCSC" "C52923" (id 4) (at 59.69 125.095 0)
       (effects (font (size 1.27 1.27)) hide)
     )
@@
       (effects (font (size 1.27 1.27)) (justify left))
     )
-    (property "Value" "2.2uF 50V" (id 1) (at 130.5561 47.5043 0)
+    (property "Value" "1uF 25v" (id 1) (at 130.5561 47.5043 0)
       (effects (font (size 1.27 1.27)) (justify left))
     )
@@
       (effects (font (size 1.27 1.27)) hide)
     )
-    (property "LCSC" "C50254" (id 4) (at 127.635 46.355 0)
+    (property "LCSC" "C52923" (id 4) (at 127.635 46.355 0)
       (effects (font (size 1.27 1.27)) hide)
     )
@@
       (effects (font (size 1.27 1.27)) (justify left))
     )
-    (property "Value" "2.2uF 50V" (id 1) (at 155.9561 104.6543 0)
+    (property "Value" "1uF 25v" (id 1) (at 155.9561 104.6543 0)
       (effects (font (size 1.27 1.27)) (justify left))
     )
@@
       (effects (font (size 1.27 1.27)) hide)
     )
-    (property "LCSC" "C50254" (id 4) (at 153.035 103.505 0)
+    (property "LCSC" "C52923" (id 4) (at 153.035 103.505 0)
       (effects (font (size 1.27 1.27)) hide)
     )
@@
       (effects (font (size 1.27 1.27)) (justify left))
     )
-    (property "Value" "2.2uF 50V" (id 1) (at 155.9561 156.0893 0)
+    (property "Value" "1uF 25v" (id 1) (at 155.9561 156.0893 0)
       (effects (font (size 1.27 1.27)) (justify left))
     )
@@
       (effects (font (size 1.27 1.27)) hide)
     )
-    (property "LCSC" "C50254" (id 4) (at 153.035 154.94 0)
+    (property "LCSC" "C52923" (id 4) (at 153.035 154.94 0)
       (effects (font (size 1.27 1.27)) hide)
     )
@@
       (effects (font (size 1.27 1.27)) (justify left))
     )
-    (property "Value" "2.2uF 50V" (id 1) (at 218.8211 124.9743 0)
+    (property "Value" "1uF 25v" (id 1) (at 218.8211 124.9743 0)
       (effects (font (size 1.27 1.27)) (justify left))
     )
@@
       (effects (font (size 1.27 1.27)) hide)
     )
-    (property "LCSC" "C50254" (id 4) (at 229.235 121.92 0)
+    (property "LCSC" "C52923" (id 4) (at 229.235 121.92 0)
       (effects (font (size 1.27 1.27)) hide)
     )
@@
       (effects (font (size 1.27 1.27)) (justify left))
     )
-    (property "Value" "2.2uF 50V" (id 1) (at 253.1111 90.6843 0)
+    (property "Value" "1uF 25v" (id 1) (at 253.1111 90.6843 0)
       (effects (font (size 1.27 1.27)) (justify left))
     )
@@
       (effects (font (size 1.27 1.27)) hide)
     )
-    (property "LCSC" "C50254" (id 4) (at 250.19 89.535 0)
+    (property "LCSC" "C52923" (id 4) (at 250.19 89.535 0)
       (effects (font (size 1.27 1.27)) hide)
     )
@@
     )
     (path "/f86e3d36-fa27-4c5c-91fd-77ed15b7c591"
-      (reference "C1") (unit 1) (value "2.2uF 50V") (footprint "Capacitor_SMD:C_0402_1005Metric")
+      (reference "C1") (unit 1) (value "1uF 25v") (footprint "Capacitor_SMD:C_0402_1005Metric")
     )
     (path "/69fd1c5a-6f09-4a27-bad7-163f2cd45b60"
-      (reference "C2") (unit 1) (value "2.2uF 50V") (footprint "Capacitor_SMD:C_0402_1005Metric")
+      (reference "C2") (unit 1) (value "1uF 25v") (footprint "Capacitor_SMD:C_0402_1005Metric")
     )
     (path "/66be52dd-1925-4762-912a-17f2ff76de53"
-      (reference "C3") (unit 1) (value "2.2uF 50V") (footprint "Capacitor_SMD:C_0402_1005Metric")
+      (reference "C3") (unit 1) (value "1uF 25v") (footprint "Capacitor_SMD:C_0402_1005Metric")
     )
     (path "/85e8bbdc-1d1f-44b6-b2fc-75b9a8e53e90"
-      (reference "C4") (unit 1) (value "2.2uF 50V") (footprint "Capacitor_SMD:C_0402_1005Metric")
+      (reference "C4") (unit 1) (value "1uF 25v") (footprint "Capacitor_SMD:C_0402_1005Metric")
     )
     (path "/103facbe-016e-4ec9-bd2b-f2db43a64fc6"
@@
     )
     (path "/842b5d71-620f-438b-94c4-e714de61b21d"
-      (reference "C8") (unit 1) (value "2.2uF 50V") (footprint "Capacitor_SMD:C_0402_1005Metric")
+      (reference "C8") (unit 1) (value "1uF 25v") (footprint "Capacitor_SMD:C_0402_1005Metric")
     )
     (path "/707a1c10-d803-4cb8-8475-c265c3d63d07"
-      (reference "C9") (unit 1) (value "2.2uF 50V") (footprint "Capacitor_SMD:C_0402_1005Metric")
+      (reference "C9") (unit 1) (value "1uF 25v") (footprint "Capacitor_SMD:C_0402_1005Metric")
     )
     (path "/ff248a56-67cb-4e99-b51f-78c47141cc03"
