File: beetledouble/driver.kicad_sch (KiCad schematic)
At the start: 19 parts, among them J4 motor_out, Q1 AON6884, Q2 AON6884, U4 NCP81155MN, U5 NCP81155MN

Commit message: Updates
Parts:
- C3, C4: LCSC C326557 -> C162273
- J4: footprint Connector_Wire:SolderWire-0.75sqmm_1x02_P4.8mm_D1.25mm_OD2.3mm -> beetledouble:beetlemotor
- Q1, Q2: value AON6884 -> SE3082G; LCSC C125872 -> C238670
Other:
- note added: "Chinese part: SINO-IC SE3082G"
- note added: "Previous part: AON6884 (became unavailable)"
- note added: "Total gate charge - approx 50 nC (Datasheet: 50nC typ) Q = 5e-8 at 10 volts, a 1uF capacitor stores 10x 1e-6 = 1e-5 C"
- note removed: "Total gate charge - approx 10 nC (Datasheet: 9nC max) at 10 volts, a 1uF capacitor stores 10x 1e-6 = 1e-5 C So enough for at least 100 charges."
Changed lines of the file:
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@@
     (effects (font (size 1.27 1.27)) (justify right bottom))
   )
-  (text "Total gate charge - approx 10 nC (Datasheet: 9nC max)\n\nat 10 volts, a 1uF capacitor stores 10x 1e-6 = 1e-5 C \nSo enough for at least 100 charges."
+  (text "Total gate charge - approx 50 nC (Datasheet: 50nC typ)\nQ = 5e-8\n\nat 10 volts, a 1uF capacitor stores 10x 1e-6 = 1e-5 C \n"
     (at 154.94 29.845 0)
     (effects (font (size 1.27 1.27)) (justify right bottom))
@@
   (text "H-Bridge\n" (at 227.33 70.485 180)
     (effects (font (size 1.27 1.27)) (justify right bottom))
+  )
+  (text "Previous part: AON6884 (became unavailable)" (at 229.235 49.53 0)
+    (effects (font (size 1.27 1.27)) (justify left bottom))
+  )
+  (text "Chinese part:\nSINO-IC SE3082G" (at 229.87 55.88 0)
+    (effects (font (size 1.27 1.27)) (justify left bottom))
   )
   (label "MOTORH1" (at 71.755 96.52 180)
@@
       (effects (font (size 1.27 1.27)) (justify right))
     )
-    (property "Footprint" "Connector_Wire:SolderWire-0.75sqmm_1x02_P4.8mm_D1.25mm_OD2.3mm" (id 2) (at 231.775 78.105 0)
+    (property "Footprint" "beetledouble:beetlemotor" (id 2) (at 231.775 78.105 0)
       (effects (font (size 1.27 1.27)) hide)
     )
@@
       (effects (font (size 1.27 1.27)) hide)
     )
-    (property "LCSC" "C326557" (id 4) (at 73.66 87.63 0)
+    (property "LCSC" "C162273" (id 4) (at 73.66 87.63 0)
       (effects (font (size 1.27 1.27)) hide)
     )
@@
       (effects (font (size 1.27 1.27)) hide)
     )
-    (property "LCSC" "C326557" (id 4) (at 73.66 146.05 0)
+    (property "LCSC" "C162273" (id 4) (at 73.66 146.05 0)
       (effects (font (size 1.27 1.27)) hide)
     )
@@
       (effects (font (size 1.27 1.27)) (justify left))
     )
-    (property "Value" "AON6884" (id 1) (at 215.265 80.6449 0)
+    (property "Value" "SE3082G" (id 1) (at 215.265 80.6449 0)
       (effects (font (size 1.27 1.27)) (justify left))
     )
@@
       (effects (font (size 1.27 1.27)) hide)
     )
-    (property "LCSC" "C125872" (id 4) (at 208.28 78.74 0)
+    (property "LCSC" "C238670" (id 4) (at 208.28 78.74 0)
       (effects (font (size 1.27 1.27)) hide)
     )
@@
       (effects (font (size 1.27 1.27)) (justify left))
     )
-    (property "Value" "AON6884" (id 1) (at 214.63 93.9799 0)
+    (property "Value" "SE3082G" (id 1) (at 214.63 93.9799 0)
       (effects (font (size 1.27 1.27)) (justify left))
     )
@@
       (effects (font (size 1.27 1.27)) hide)
     )
-    (property "LCSC" "C125872" (id 4) (at 208.28 92.075 0)
+    (property "LCSC" "C238670" (id 4) (at 208.28 92.075 0)
       (effects (font (size 1.27 1.27)) hide)
     )
@@
       (effects (font (size 1.27 1.27)) (justify left))
     )
-    (property "Value" "AON6884" (id 1) (at 263.525 80.6449 0)
+    (property "Value" "SE3082G" (id 1) (at 263.525 80.6449 0)
       (effects (font (size 1.27 1.27)) (justify left))
     )
@@
       (effects (font (size 1.27 1.27)) hide)
     )
-    (property "LCSC" "C125872" (id 4) (at 256.54 78.74 0)
+    (property "LCSC" "C238670" (id 4) (at 256.54 78.74 0)
       (effects (font (size 1.27 1.27)) hide)
     )
@@
       (effects (font (size 1.27 1.27)) (justify left))
     )
-    (property "Value" "AON6884" (id 1) (at 262.89 93.9799 0)
+    (property "Value" "SE3082G" (id 1) (at 262.89 93.9799 0)
       (effects (font (size 1.27 1.27)) (justify left))
     )
@@
       (effects (font (size 1.27 1.27)) hide)
     )
-    (property "LCSC" "C125872" (id 4) (at 256.54 92.075 0)
-      (effects (font (size 1.27 1.27)) hide)
-    )
+    (property "LCSC" "C238670" (id 4) (at 256.54 92.075 0)
+      (effects (font (size 1.27 1.27)) hide)
+    )

Commit message: Updates
Parts:
- renumbered C11 to C14, C12 to C15, C13 to C16, C17 to C18, C3 to C5, C4 to C6, D3 to D5, D4 to D6, J4 to J5, Q1 to Q3, Q2 to Q4, R1 to R5, R2 to R6, R3 to R7, R4 to R8, U4 to U6, U5 to U7
Changed lines of the file:
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@@
   (symbol (lib_id "power:+12V") (at 52.705 72.39 0)
     (in_bom yes) (on_board yes)
-    (property "Reference" "#PWR08" (id 0) (at 52.705 76.2 0)
+    (property "Reference" "#PWR012" (id 0) (at 52.705 76.2 0)
       (effects (font (size 1.27 1.27)) hide)
     )
@@
   (symbol (lib_id "power:+12V") (at 52.705 135.89 0)
     (in_bom yes) (on_board yes)
-    (property "Reference" "#PWR06" (id 0) (at 52.705 139.7 0)
+    (property "Reference" "#PWR010" (id 0) (at 52.705 139.7 0)
       (effects (font (size 1.27 1.27)) hide)
     )
@@
   (symbol (lib_id "power:GND") (at 52.705 115.57 0)
     (in_bom yes) (on_board yes)
-    (property "Reference" "#PWR09" (id 0) (at 52.705 121.92 0)
+    (property "Reference" "#PWR013" (id 0) (at 52.705 121.92 0)
       (effects (font (size 1.27 1.27)) hide)
     )
@@
   (symbol (lib_id "power:GND") (at 52.705 177.165 0)
     (in_bom yes) (on_board yes)
-    (property "Reference" "#PWR07" (id 0) (at 52.705 183.515 0)
+    (property "Reference" "#PWR011" (id 0) (at 52.705 183.515 0)
       (effects (font (size 1.27 1.27)) hide)
     )
@@
   (symbol (lib_id "Device:R") (at 80.01 154.94 90)
     (in_bom yes) (on_board yes)
-    (property "Reference" "R1" (id 0) (at 80.01 149.7138 90))
+    (property "Reference" "R5" (id 0) (at 80.01 149.7138 90))
     (property "Value" "10R" (id 1) (at 80.01 152.0125 90))
     (property "Footprint" "Resistor_SMD:R_0603_1608Metric" (id 2) (at 80.01 156.718 90)
@@
   (symbol (lib_id "Device:R") (at 80.01 162.56 90)
     (in_bom yes) (on_board yes)
-    (property "Reference" "R2" (id 0) (at 80.01 157.3338 90))
+    (property "Reference" "R6" (id 0) (at 80.01 157.3338 90))
     (property "Value" "10R" (id 1) (at 80.01 159.6325 90))
     (property "Footprint" "Resistor_SMD:R_0603_1608Metric" (id 2) (at 80.01 164.338 90)
@@
   (symbol (lib_id "Device:R") (at 83.185 96.52 90)
     (in_bom yes) (on_board yes)
-    (property "Reference" "R3" (id 0) (at 83.185 91.2938 90))
+    (property "Reference" "R7" (id 0) (at 83.185 91.2938 90))
     (property "Value" "10R" (id 1) (at 83.185 93.5925 90))
     (property "Footprint" "Resistor_SMD:R_0603_1608Metric" (id 2) (at 83.185 98.298 90)
@@
   (symbol (lib_id "Device:R") (at 83.185 104.14 90)
     (in_bom yes) (on_board yes)
-    (property "Reference" "R4" (id 0) (at 83.185 98.9138 90))
+    (property "Reference" "R8" (id 0) (at 83.185 98.9138 90))
     (property "Value" "10R" (id 1) (at 83.185 101.2125 90))
     (property "Footprint" "Resistor_SMD:R_0603_1608Metric" (id 2) (at 83.185 105.918 90)
@@
   (symbol (lib_id "Connector:Conn_01x02_Female") (at 231.775 78.105 90)
     (in_bom yes) (on_board yes)
-    (property "Reference" "J4" (id 0) (at 236.4487 79.648 90)
+    (property "Reference" "J5" (id 0) (at 236.4487 79.648 90)
       (effects (font (size 1.27 1.27)) (justify right))
     )
@@
   (symbol (lib_id "Device:D_Schottky") (at 56.515 80.01 180)
     (in_bom yes) (on_board yes) (fields_autoplaced)
-    (property "Reference" "D3" (id 0) (at 56.515 74.93 0))
+    (property "Reference" "D5" (id 0) (at 56.515 74.93 0))
     (property "Value" "B5819W" (id 1) (at 56.515 77.47 0))
     (property "Footprint" "Diode_SMD:D_SOD-123" (id 2) (at 56.515 80.01 0)
@@
   (symbol (lib_id "Device:D_Schottky") (at 59.055 139.7 180)
     (in_bom yes) (on_board yes) (fields_autoplaced)
-    (property "Reference" "D4" (id 0) (at 59.055 134.62 0))
+    (property "Reference" "D6" (id 0) (at 59.055 134.62 0))
     (property "Value" "B5819W" (id 1) (at 59.055 137.16 0))
     (property "Footprint" "Diode_SMD:D_SOD-123" (id 2) (at 59.055 139.7 0)
@@
   (symbol (lib_id "Device:C") (at 73.66 87.63 0)
     (in_bom yes) (on_board yes)
-    (property "Reference" "C3" (id 0) (at 76.5811 86.4806 0)
+    (property "Reference" "C5" (id 0) (at 76.5811 86.4806 0)
       (effects (font (size 1.27 1.27)) (justify left))
     )
@@
   (symbol (lib_id "Device:C") (at 73.66 146.05 0)
     (in_bom yes) (on_board yes)
-    (property "Reference" "C4" (id 0) (at 76.581 144.901 0)
+    (property "Reference" "C6" (id 0) (at 76.581 144.901 0)
       (effects (font (size 1.27 1.27)) (justify left))
     )
@@
   (symbol (lib_id "Device:C") (at 158.75 85.09 0)
     (in_bom yes) (on_board yes)
-    (property "Reference" "C11" (id 0) (at 161.6711 83.9406 0)
+    (property "Reference" "C14" (id 0) (at 161.6711 83.9406 0)
       (effects (font (size 1.27 1.27)) (justify left))
     )
@@
   (symbol (lib_id "Device:C") (at 170.18 85.09 0)
     (in_bom yes) (on_board yes)
-    (property "Reference" "C12" (id 0) (at 173.1011 83.9406 0)
+    (property "Reference" "C15" (id 0) (at 173.1011 83.9406 0)
       (effects (font (size 1.27 1.27)) (justify left))
     )
@@
   (symbol (lib_id "Device:C") (at 179.705 85.09 0)
     (in_bom yes) (on_board yes)
-    (property "Reference" "C13" (id 0) (at 180.0861 82.6706 0)
+    (property "Reference" "C16" (id 0) (at 180.0861 82.6706 0)
       (effects (font (size 1.27 1.27)) (justify left))
     )
@@
   (symbol (lib_id "Device:C") (at 186.055 85.09 0)
     (in_bom yes) (on_board yes)
-    (property "Reference" "C17" (id 0) (at 187.0711 82.0356 0)
+    (property "Reference" "C18" (id 0) (at 187.0711 82.0356 0)
       (effects (font (size 1.27 1.27)) (justify left))
     )
@@
   (symbol (lib_id "Device:Q_Dual_PMOS_S1G1S2G2D2D2D1D1") (at 208.28 78.74 0)
     (in_bom yes) (on_board yes) (fields_autoplaced)
-    (property "Reference" "Q1" (id 0) (at 215.265 78.1049 0)
+    (property "Reference" "Q3" (id 0) (at 215.265 78.1049 0)
       (effects (font (size 1.27 1.27)) (justify left))
     )
@@
   (symbol (lib_id "Device:Q_Dual_PMOS_S1G1S2G2D2D2D1D1") (at 208.28 92.075 0)
     (in_bom yes) (on_board yes) (fields_autoplaced)
-    (property "Reference" "Q1" (id 0) (at 214.63 91.4399 0)
+    (property "Reference" "Q3" (id 0) (at 214.63 91.4399 0)
       (effects (font (size 1.27 1.27)) (justify left))
     )
@@
     )
     (property "LCSC" "C238670" (id 4) (at 208.28 92.075 0)
-      (effects (font (size 1.27 1.27)) hide)
-    )
-    (pin "3")
-    (pin "4")
-    (pin "5")
-    (pin "6")
-  )
-  (symbol (lib_id "Device:Q_Dual_PMOS_S1G1S2G2D2D2D1D1") (at 256.54 78.74 0)
-    (in_bom yes) (on_board yes) (fields_autoplaced)
-    (property "Reference" "Q2" (id 0) (at 263.525 78.1049 0)
-      (effects (font (size 1.27 1.27)) (justify left))
-    )
-    (property "Value" "SE3082G" (id 1) (at 263.525 80.6449 0)
-      (effects (font (size 1.27 1.27)) (justify left))
-    )
-    (property "Footprint" "beetledouble:Infineon-PG-TDSON" (id 2) (at 257.81 78.74 0)
-      (effects (font (size 1.27 1.27)) hide)
-    )
-    (property "Datasheet" "~" (id 3) (at 257.81 78.74 0)
-      (effects (font (size 1.27 1.27)) hide)
-    )
-    (property "LCSC" "C238670" (id 4) (at 256.54 78.74 0)
       (effects (font (size 1.27 1.27)) hide)
     )
@@
     (pin "8")
   )
+  (symbol (lib_id "Device:Q_Dual_PMOS_S1G1S2G2D2D2D1D1") (at 256.54 78.74 0)
+    (in_bom yes) (on_board yes) (fields_autoplaced)
+    (property "Reference" "Q4" (id 0) (at 263.525 78.1049 0)
+      (effects (font (size 1.27 1.27)) (justify left))
+    )
+    (property "Value" "SE3082G" (id 1) (at 263.525 80.6449 0)
+      (effects (font (size 1.27 1.27)) (justify left))
+    )
+    (property "Footprint" "beetledouble:Infineon-PG-TDSON" (id 2) (at 257.81 78.74 0)
+      (effects (font (size 1.27 1.27)) hide)
+    )
+    (property "Datasheet" "~" (id 3) (at 257.81 78.74 0)
+      (effects (font (size 1.27 1.27)) hide)
+    )
+    (property "LCSC" "C238670" (id 4) (at 256.54 78.74 0)
+      (effects (font (size 1.27 1.27)) hide)
+    )
+    (pin "1")
+    (pin "2")
+    (pin "7")
+    (pin "8")
+  )
   (symbol (lib_id "Device:Q_Dual_PMOS_S1G1S2G2D2D2D1D1") (at 256.54 92.075 0)
     (in_bom yes) (on_board yes) (fields_autoplaced)
-    (property "Reference" "Q2" (id 0) (at 262.89 91.4399 0)
+    (property "Reference" "Q4" (id 0) (at 262.89 91.4399 0)
       (effects (font (size 1.27 1.27)) (justify left))
     )
@@
       (effects (font (size 1.27 1.27)) hide)
     )
-    (pin "3")
-    (pin "4")
-    (pin "5")
-    (pin "6")
+    (pin "1")
+    (pin "2")
+    (pin "7")
+    (pin "8")
   )
   (symbol (lib_id "beetledouble:NCP81155MN") (at 52.705 100.33 0)
     (in_bom yes) (on_board yes)
-    (property "Reference" "U4" (id 0) (at 44.1325 90.17 0))
+    (property "Reference" "U6" (id 0) (at 44.1325 90.17 0))
     (property "Value" "NCP81155MN" (id 1) (at 44.1325 87.63 0))
     (property "Footprint" "beetledouble:DFN-8-3x3mm_hand1" (id 2) (at 52.705 100.33 0)
@@
   (symbol (lib_id "beetledouble:NCP81155MN") (at 52.705 158.75 0)
     (in_bom yes) (on_board yes)
-    (property "Reference" "U5" (id 0) (at 44.1325 148.59 0))
+    (property "Reference" "U7" (id 0) (at 44.1325 148.59 0))
     (property "Value" "NCP81155MN" (id 1) (at 44.1325 146.05 0))
     (property "Footprint" "beetledouble:DFN-8-3x3mm_hand1" (id 2) (at 52.705 158.75 0)
