File: beetleback_cg2/beetleback_cg2.kicad_pcb (KiCad board)
At the start: 4 copper layers, 44 x 35.5 mm, 33 parts, among them J1 signalin, J2 powerin, J3 motor_pad_1, J4 motor_pad_2, Q1 IRF8313PBF, Q2 IRF8313PBF, U1 ATtiny13A-SS, U2 ADP3110A, U3 HT7550-2, U4 ADP3110A, U5 HT75C0-2

Commit message: edge rails
Parts:
- added REF**: jlc_toolhole, beetleback:jlc_toolhole, B.Cu at (74.1, 136.0)
- added REF**: mousebites, beetleback:mousebites, B.Cu at (78.1, 113.5)
- added REF**: mousebites, beetleback:mousebites, B.Cu at (78.1, 124.5)
- added REF**: jlc_toolhole, beetleback:jlc_toolhole, B.Cu at (74.1, 111.0)
- moved REF** 16.2 mm to (101.1, 113.5)
- moved REF** 16.2 mm to (105.1, 111.0)
- moved REF** 16.2 mm to (101.1, 124.5)
- moved REF** 16.2 mm to (105.1, 136.0)
- moved C2 4.00 mm to (100.4, 120.5)
Routing:
- net /MOTOR_PAD_2: track 30.7 -> 33.7 mm
- added copper zone on B.Cu, net (none)
- added copper zone on F.Cu, net (none)
Other:
- board size 44 x 35.5 mm -> 35 x 35.5 mm
- board text removed: "ACTIVE"

Commit message: update
Parts:
- removed the REF** at (105.1, 111.0)
- removed the REF** at (105.1, 136.0)
- removed the REF** at (74.1, 136.0)
- removed the REF** at (74.1, 111.0)
- J2: footprint Connector_Wire:SolderWire-1sqmm_1x02_P5.4mm_D1.4mm_OD2.7mm -> beetleback:beetlepower_in
- REF** (x2): moved to F.Cu
- moved U5 2.75 mm to (85.3, 119.2)
- moved C1 2.51 mm to (84.8, 122.0)
- moved C5 1.75 mm to (81.1, 122.5)
- moved C6 1.75 mm to (81.1, 120.2)
- moved C7 1.75 mm to (81.1, 118.0)
- moved D3 0.56 mm to (85.3, 127.0)
Connections:
- net Net-(R4-Pad1) renamed /BLINKY
Routing:
- net +5V: track 17.3 -> 20.2 mm
- net /VBAT: track 40.8 -> 42.4 mm, vias 12 -> 14
- net GND: track 45.6 -> 44.1 mm, vias 13 -> 15
- net /GH2: track 19.8 -> 19.2 mm
Other:
- board text added: "Tool hole strip"
- board text removed: "12"
- board text removed: "5"

Commit message: tweaks
Parts:
- J1: footprint Connector_PinHeader_2.54mm:PinHeader_1x03_P2.54mm_Vertical -> beetleback:rx_pins
Other:
- board text added: "12"
- board text added: "5"
- board text added: "G"
Changed lines of the file:
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@@
-(kicad_pcb (version 20210623) (generator pcbnew)
+(kicad_pcb (version 20210722) (generator pcbnew)
   (general
     (thickness 1.6)
@@
   (setup
     (stackup
-      (layer "F.SilkS" (type "Top Silk Screen"))
+      (layer "F.SilkS" (type "Top Silk Screen") (color "White"))
       (layer "F.Paste" (type "Top Solder Paste"))
       (layer "F.Mask" (type "Top Solder Mask") (color "Green") (thickness 0.01))
@@
       (layer "B.Mask" (type "Bottom Solder Mask") (color "Green") (thickness 0.01))
       (layer "B.Paste" (type "Bottom Solder Paste"))
-      (layer "B.SilkS" (type "Bottom Silk Screen"))
+      (layer "B.SilkS" (type "Bottom Silk Screen") (color "White"))
       (copper_finish "None")
       (dielectric_constraints no)
@@
     )
   )
-  (footprint "Connector_PinHeader_2.54mm:PinHeader_1x03_P2.54mm_Vertical" (layer "F.Cu")
+  (footprint "beetleback:rx_pins" (layer "F.Cu")
     (at 98.625 111.5 -90)
     (descr "Through hole straight pin header, 1x03, 2.54mm pitch, single row")
@@
       (effects (font (size 1 1) (thickness 0.15)))
     )
-    (fp_line (start 1.33 1.27) (end 1.33 6.41) (layer "F.SilkS") (width 0.12))
-    (fp_line (start -1.33 -1.33) (end 0 -1.33) (layer "F.SilkS") (width 0.12))
-    (fp_line (start -1.33 1.27) (end -1.33 6.41) (layer "F.SilkS") (width 0.12))
-    (fp_line (start -1.33 1.27) (end 1.33 1.27) (layer "F.SilkS") (width 0.12))
-    (fp_line (start -1.33 0) (end -1.33 -1.33) (layer "F.SilkS") (width 0.12))
-    (fp_line (start -1.33 6.41) (end 1.33 6.41) (layer "F.SilkS") (width 0.12))
+    (fp_line (start -1.8 -1.8) (end -1.8 6.85) (layer "F.CrtYd") (width 0.05))
     (fp_line (start -1.8 6.85) (end 1.8 6.85) (layer "F.CrtYd") (width 0.05))
+    (fp_line (start 1.8 -1.8) (end -1.8 -1.8) (layer "F.CrtYd") (width 0.05))
     (fp_line (start 1.8 6.85) (end 1.8 -1.8) (layer "F.CrtYd") (width 0.05))
-    (fp_line (start 1.8 -1.8) (end -1.8 -1.8) (layer "F.CrtYd") (width 0.05))
-    (fp_line (start -1.8 -1.8) (end -1.8 6.85) (layer "F.CrtYd") (width 0.05))
+    (fp_line (start 1.27 -1.27) (end 1.27 6.35) (layer "F.Fab") (width 0.1))
+    (fp_line (start -1.27 6.35) (end -1.27 -0.635) (layer "F.Fab") (width 0.1))
+    (fp_line (start 1.27 6.35) (end -1.27 6.35) (layer "F.Fab") (width 0.1))
+    (fp_line (start -0.635 -1.27) (end 1.27 -1.27) (layer "F.Fab") (width 0.1))
     (fp_line (start -1.27 -0.635) (end -0.635 -1.27) (layer "F.Fab") (width 0.1))
-    (fp_line (start 1.27 6.35) (end -1.27 6.35) (layer "F.Fab") (width 0.1))
-    (fp_line (start 1.27 -1.27) (end 1.27 6.35) (layer "F.Fab") (width 0.1))
-    (fp_line (start -0.635 -1.27) (end 1.27 -1.27) (layer "F.Fab") (width 0.1))
-    (fp_line (start -1.27 6.35) (end -1.27 -0.635) (layer "F.Fab") (width 0.1))
-    (pad "1" thru_hole rect locked (at 0 0 270) (size 1.7 1.7) (drill 1) (layers *.Cu *.Mask)
-      (net 20 "/PWMIN1") (pinfunction "Pin_1") (pintype "passive"))
-    (pad "2" thru_hole oval locked (at 0 2.54 270) (size 1.7 1.7) (drill 1) (layers *.Cu *.Mask)
-      (net 16 "+5V") (pinfunction "Pin_2") (pintype "passive"))
-    (pad "3" thru_hole oval locked (at 0 5.08 270) (size 1.7 1.7) (drill 1) (layers *.Cu *.Mask)
-      (net 7 "GND") (pinfunction "Pin_3") (pintype "passive"))
+    (pad "1" thru_hole rect (at 0 0 270) (size 1.8 1.8) (drill 1.2) (layers *.Cu *.Mask)
+      (net 20 "/PWMIN1") (pinfunction "Pin_1"))
+    (pad "2" thru_hole oval (at 0 2.54 270) (size 1.8 1.8) (drill 1.2) (layers *.Cu *.Mask)
+      (net 16 "+5V") (pinfunction "Pin_2"))
+    (pad "3" thru_hole oval (at 0 5.08 270) (size 1.8 1.8) (drill 1.2) (layers *.Cu *.Mask)
+      (net 7 "GND") (pinfunction "Pin_3"))
     (model "${KICAD6_3DMODEL_DIR}/Connector_PinHeader_2.54mm.3dshapes/PinHeader_1x03_P2.54mm_Vertical.wrl"
       (offset (xyz 0 0 0))
@@
   (gr_circle (center 90.1 138.5) (end 90.6 138.5) (layer "F.SilkS") (width 0.12) (fill solid))
   (gr_circle (center 89.6 133.5) (end 93.6 133.5) (layer "F.SilkS") (width 0.12) (fill none))
+  (gr_line (start 87.6 144) (end 88.1 143.5) (layer "F.SilkS") (width 0.12))
   (gr_circle (center 84.1 123.75) (end 84.6 123.75) (layer "F.SilkS") (width 0.12) (fill solid))
+  (gr_line (start 87.6 144) (end 88.1 144.5) (layer "F.SilkS") (width 0.12))
   (gr_circle (center 88.6 127) (end 89.1 127) (layer "F.SilkS") (width 0.12) (fill solid))
   (gr_circle (center 100.6 128) (end 101.1 128) (layer "F.SilkS") (width 0.12) (fill solid))
-  (gr_circle (center 88.6 144) (end 89.1 144) (layer "F.SilkS") (width 0.12) (fill solid))
+  (gr_line (start 89.6 144) (end 87.6 144) (layer "F.SilkS") (width 0.12))
   (gr_line (start 89.6 133.5) (end 89.6 156) (layer "Dwgs.User") (width 0.1))
   (gr_line (start 97.15 131.25) (end 82.05 135.75) (layer "Dwgs.User") (width 0.1))
@@
     (effects (font (size 1 1) (thickness 0.15)) (justify mirror))
   )
+  (gr_text "12" (at 87.6 119.5 90) (layer "F.SilkS")
+    (effects (font (size 0.8 0.8) (thickness 0.15)))
+  )
   (gr_text "-" (at 85.6 117) (layer "F.SilkS")
     (effects (font (size 1 1) (thickness 0.15)))
@@
     (effects (font (size 1 1) (thickness 0.15)))
   )
+  (gr_text "G" (at 93.5 112.6 270) (layer "F.SilkS")
+    (effects (font (size 1 1) (thickness 0.15)) (justify left))
+  )
   (gr_text "-" (at 88.1 115.5 90) (layer "F.SilkS")
     (effects (font (size 1 1) (thickness 0.15)))
@@
     (effects (font (size 1 1) (thickness 0.15)))
   )
-  (gr_text "RX" (at 98.6 113 270) (layer "F.SilkS")
+  (gr_text "RX" (at 98.6 112.6 270) (layer "F.SilkS")
     (effects (font (size 1 1) (thickness 0.15)) (justify left))
   )
-  (gr_text "+5" (at 96.1 113 270) (layer "F.SilkS")
+  (gr_text "+5" (at 96.1 112.6 270) (layer "F.SilkS")
     (effects (font (size 1 1) (thickness 0.15)) (justify left))
+  )
+  (gr_text "5" (at 90.1 115) (layer "F.SilkS")
+    (effects (font (size 0.8 0.8) (thickness 0.15)))
   )
   (gr_text "MCU" (at 87.1 123.25 90) (layer "F.SilkS")
     (effects (font (size 0.8 0.8) (thickness 0.15)))
   )
-  (gr_text "JLC: Different net clearance: 0.127, use 0.15 to be sure" (at 84.8 105.9) (layer "Dwgs.User")
+  (gr_text "JLC: Different net clearance: 0.127, use 0.15 to be sure" (at 84.8 87) (layer "Dwgs.User")
     (effects (font (size 1.5 1.5) (thickness 0.3)))
   )
-  (gr_text "JLC: via size (min) 0.2mm" (at 88.1 102) (layer "Dwgs.User")
+  (gr_text "JLC: via size (min) 0.2mm" (at 88.1 96) (layer "Dwgs.User")
     (effects (font (size 1 1) (thickness 0.15)))
   )
-  (gr_text "JLC: min trace with 0.15mm any layer" (at 92.85 99.5) (layer "Dwgs.User")
+  (gr_text "JLC: min trace with 0.15mm any layer" (at 92.85 93) (layer "Dwgs.User")
     (effects (font (size 1 1) (thickness 0.15)))
   )
@@
   (segment (start 98.11 117) (end 99.0625 117) (width 0.15) (layer "F.Cu") (net 17))
   (segment (start 99.0625 117) (end 99.6 117.5375) (width 0.15) (layer "F.Cu") (net 17))
-  (segment (start 80.465 125.290312) (end 82.054832 123.70048) (width 0.15) (layer "F.Cu") (net 19))
   (segment (start 89.074031 122.775969) (end 90.710454 121.139546) (width 0.15) (layer "F.Cu") (net 19))
   (segment (start 95.6 123.75) (end 96.465 122.885) (width 0.15) (layer "F.Cu") (net 19))
   (segment (start 91.6 118.5) (end 92.505 119.405) (width 0.15) (layer "F.Cu") (net 19))
+  (segment (start 80.465 125.135) (end 81.89952 123.70048) (width 0.15) (layer "F.Cu") (net 19))
   (segment (start 89.074031 122.775969) (end 85.024511 122.775969) (width 0.15) (layer "F.Cu") (net 19))
   (segment (start 85.024511 122.775969) (end 84.1 123.70048) (width 0.15) (layer "F.Cu") (net 19))
   (segment (start 96.465 122.885) (end 96.465 122.025) (width 0.15) (layer "F.Cu") (net 19))
   (segment (start 92.505 120.025) (end 92.505 121.03) (width 0.15) (layer "F.Cu") (net 19))
-  (segment (start 80.465 125.525) (end 80.465 125.290312) (width 0.15) (layer "F.Cu") (net 19))
+  (segment (start 84.1 123.70048) (end 81.89952 123.70048) (width 0.15) (layer "F.Cu") (net 19))
   (segment (start 90.710454 121.139546) (end 90.710454 119.044858) (width 0.15) (layer "F.Cu") (net 19))
+  (segment (start 80.465 125.525) (end 80.465 125.135) (width 0.15) (layer "F.Cu") (net 19))
   (segment (start 90.710454 119.044858) (end 91.255312 118.5) (width 0.15) (layer "F.Cu") (net 19))
   (segment (start 95.225 123.75) (end 95.6 123.75) (width 0.15) (layer "F.Cu") (net 19))
@@
   (segment (start 92.505 121.03) (end 95.225 123.75) (width 0.15) (layer "F.Cu") (net 19))
   (segment (start 92.505 119.405) (end 92.505 120.025) (width 0.15) (layer "F.Cu") (net 19))
-  (segment (start 82.39952 123.70048) (end 82.30048 123.70048) (width 0.15) (layer "F.Cu") (net 19))
-  (segment (start 82.054832 123.70048) (end 82.39952 123.70048) (width 0.15) (layer "F.Cu") (net 19))
-  (segment (start 84.1 123.70048) (end 82.39952 123.70048) (width 0.15) (layer "F.Cu") (net 19))
   (segment (start 98.625 115.235) (end 98.11 115.75) (width 0.15) (layer "F.Cu") (net 20))
   (segment (start 98.625 111.5) (end 98.625 115.235) (width 0.15) (layer "F.Cu") (net 20))

Commit message: old ideas
Parts:
- U5: value HT75C0-2 -> HT75C0-3
Changed lines of the file:
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@@
     (descr "SOIC, 8 Pin (JEDEC MS-012AA, https://www.analog.com/media/en/package-pcb-resources/package/pkg_pdf/soic_narrow-r/r_8.pdf), generated with kicad-footprint-generator ipc_gullwing_generator.py")
     (tags "SOIC SO")
-    (property "LCSC" "C14075")
+    (property "LCSC" "C40382")
     (property "Sheetfile" "beetleback_cg2.kicad_sch")
     (property "Sheetname" "")
@@
     (fp_line (start -1.27 -0.635) (end -0.635 -1.27) (layer "F.Fab") (width 0.1))
     (pad "1" thru_hole rect (at 0 0 270) (size 1.8 1.8) (drill 1.2) (layers *.Cu *.Mask)
-      (net 20 "/PWMIN1") (pinfunction "Pin_1"))
+      (net 20 "/PWMIN1") (pinfunction "Pin_1") (pintype "passive"))
     (pad "2" thru_hole oval (at 0 2.54 270) (size 1.8 1.8) (drill 1.2) (layers *.Cu *.Mask)
-      (net 16 "+5V") (pinfunction "Pin_2"))
+      (net 16 "+5V") (pinfunction "Pin_2") (pintype "passive"))
     (pad "3" thru_hole oval (at 0 5.08 270) (size 1.8 1.8) (drill 1.2) (layers *.Cu *.Mask)
-      (net 7 "GND") (pinfunction "Pin_3"))
+      (net 7 "GND") (pinfunction "Pin_3") (pintype "passive"))
     (model "${KICAD6_3DMODEL_DIR}/Connector_PinHeader_2.54mm.3dshapes/PinHeader_1x03_P2.54mm_Vertical.wrl"
       (offset (xyz 0 0 0))
@@
     (descr "SOT, 5 Pin (https://www.jedec.org/sites/default/files/docs/Mo-178c.PDF variant AA), generated with kicad-footprint-generator ipc_gullwing_generator.py")
     (tags "SOT TO_SOT_SMD")
-    (property "LCSC" "C95005")
+    (property "LCSC" "C259861")
     (property "Sheetfile" "beetleback_cg2.kicad_sch")
     (property "Sheetname" "")
@@
       (effects (font (size 1 1) (thickness 0.15)))
     )
-    (fp_text value "HT75C0-2" (at 0 2.4 90) (layer "F.Fab")
+    (fp_text value "HT75C0-3" (at 0 2.4 90) (layer "F.Fab")
       (effects (font (size 1 1) (thickness 0.15)))
     )
@@
   (gr_line (start 87.6 144) (end 88.1 144.5) (layer "F.SilkS") (width 0.12))
   (gr_circle (center 88.6 127) (end 89.1 127) (layer "F.SilkS") (width 0.12) (fill solid))
-  (gr_circle (center 100.6 128) (end 101.1 128) (layer "F.SilkS") (width 0.12) (fill solid))
   (gr_line (start 89.6 144) (end 87.6 144) (layer "F.SilkS") (width 0.12))
   (gr_line (start 89.6 133.5) (end 89.6 156) (layer "Dwgs.User") (width 0.1))
