File: beetleback_cg2/beetleback_cg2.kicad_sch (KiCad schematic)
At the start: 29 parts, among them J1 signalin, J2 powerin, J3 motor_pad_1, J4 motor_pad_2, Q1 IRF8313PBF, Q2 IRF8313PBF, U1 ATtiny13A-SS, U2 ADP3110A, U3 HT7550-2, U4 ADP3110A, U5 HT75C0-2

Commit message: update
Parts:
- J2: footprint Connector_Wire:SolderWire-1sqmm_1x02_P5.4mm_D1.4mm_OD2.7mm -> beetleback:beetlepower_in
Connections:
- net BLINKY: now reaches R4.1, U1.3 (PB4)
Other:
- moved on the sheet: D2, R4
Changed lines of the file:
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@@
     (stroke (width 0) (type solid) (color 0 0 0 0))
   )
-  (wire (pts (xy 178.435 63.5) (xy 184.15 63.5))
+  (wire (pts (xy 178.435 63.5) (xy 194.945 63.5))
     (stroke (width 0) (type solid) (color 0 0 0 0))
   )
@@
     (stroke (width 0) (type solid) (color 0 0 0 0))
   )
-  (wire (pts (xy 189.23 63.5) (xy 191.135 63.5))
+  (wire (pts (xy 200.025 63.5) (xy 201.93 63.5))
     (stroke (width 0) (type solid) (color 0 0 0 0))
   )
@@
   (label "GL2OUT" (at 163.83 168.275 180)
     (effects (font (size 1.27 1.27)) (justify right bottom))
+  )
+  (label "BLINKY" (at 180.975 63.5 0)
+    (effects (font (size 1.27 1.27)) (justify left bottom))
   )
   (label "GH1OUT" (at 180.975 109.22 180)
@@
     (pin "1")
   )
-  (symbol (lib_id "power:GND") (at 191.135 71.12 0) (unit 1)
-    (in_bom yes) (on_board yes)
-    (property "Reference" "#PWR08" (id 0) (at 191.135 77.47 0)
-      (effects (font (size 1.27 1.27)) hide)
-    )
-    (property "Value" "GND" (id 1) (at 191.2493 75.4444 0))
-    (property "Footprint" "" (id 2) (at 191.135 71.12 0)
-      (effects (font (size 1.27 1.27)) hide)
-    )
-    (property "Datasheet" "" (id 3) (at 191.135 71.12 0)
+  (symbol (lib_id "power:GND") (at 201.93 71.12 0) (unit 1)
+    (in_bom yes) (on_board yes)
+    (property "Reference" "#PWR08" (id 0) (at 201.93 77.47 0)
+      (effects (font (size 1.27 1.27)) hide)
+    )
+    (property "Value" "GND" (id 1) (at 202.0443 75.4444 0))
+    (property "Footprint" "" (id 2) (at 201.93 71.12 0)
+      (effects (font (size 1.27 1.27)) hide)
+    )
+    (property "Datasheet" "" (id 3) (at 201.93 71.12 0)
       (effects (font (size 1.27 1.27)) hide)
     )
@@
     (pin "2")
   )
-  (symbol (lib_id "Device:R_Small") (at 186.69 63.5 90) (unit 1)
-    (in_bom yes) (on_board yes)
-    (property "Reference" "R4" (id 0) (at 190.5 62.3632 90))
-    (property "Value" "1k" (id 1) (at 186.69 65.9319 90))
-    (property "Footprint" "Resistor_SMD:R_0402_1005Metric" (id 2) (at 186.69 63.5 0)
-      (effects (font (size 1.27 1.27)) hide)
-    )
-    (property "Datasheet" "~" (id 3) (at 186.69 63.5 0)
-      (effects (font (size 1.27 1.27)) hide)
-    )
-    (property "LCSC" "C11702" (id 4) (at 186.69 63.5 0)
+  (symbol (lib_id "Device:R_Small") (at 197.485 63.5 90) (unit 1)
+    (in_bom yes) (on_board yes)
+    (property "Reference" "R4" (id 0) (at 201.295 62.3632 90))
+    (property "Value" "1k" (id 1) (at 197.485 65.9319 90))
+    (property "Footprint" "Resistor_SMD:R_0402_1005Metric" (id 2) (at 197.485 63.5 0)
+      (effects (font (size 1.27 1.27)) hide)
+    )
+    (property "Datasheet" "~" (id 3) (at 197.485 63.5 0)
+      (effects (font (size 1.27 1.27)) hide)
+    )
+    (property "LCSC" "C11702" (id 4) (at 197.485 63.5 0)
       (effects (font (size 1.27 1.27)) hide)
     )
@@
     (property "Reference" "J2" (id 0) (at 19.8374 60.325 0))
     (property "Value" "powerin" (id 1) (at 25.5524 57.15 0))
-    (property "Footprint" "Connector_Wire:SolderWire-1sqmm_1x02_P5.4mm_D1.4mm_OD2.7mm" (id 2) (at 22.86 59.69 0)
+    (property "Footprint" "beetleback:beetlepower_in" (id 2) (at 22.86 59.69 0)
       (effects (font (size 1.27 1.27)) hide)
     )
@@
     (pin "2")
   )
-  (symbol (lib_id "Device:LED") (at 191.135 67.31 90) (unit 1)
-    (in_bom yes) (on_board yes)
-    (property "Reference" "D2" (id 0) (at 194.0561 66.3511 90)
+  (symbol (lib_id "Device:LED") (at 201.93 67.31 90) (unit 1)
+    (in_bom yes) (on_board yes)
+    (property "Reference" "D2" (id 0) (at 204.8511 66.3511 90)
       (effects (font (size 1.27 1.27)) (justify right))
     )
-    (property "Value" "Red LED" (id 1) (at 194.056 68.65 90)
+    (property "Value" "Red LED" (id 1) (at 204.851 68.65 90)
       (effects (font (size 1.27 1.27)) (justify right))
     )
-    (property "Footprint" "LED_SMD:LED_0603_1608Metric" (id 2) (at 191.135 67.31 0)
-      (effects (font (size 1.27 1.27)) hide)
-    )
-    (property "Datasheet" "~" (id 3) (at 191.135 67.31 0)
-      (effects (font (size 1.27 1.27)) hide)
-    )
-    (property "LCSC" "C2286" (id 4) (at 191.135 67.31 0)
+    (property "Footprint" "LED_SMD:LED_0603_1608Metric" (id 2) (at 201.93 67.31 0)
+      (effects (font (size 1.27 1.27)) hide)
+    )
+    (property "Datasheet" "~" (id 3) (at 201.93 67.31 0)
+      (effects (font (size 1.27 1.27)) hide)
+    )
+    (property "LCSC" "C2286" (id 4) (at 201.93 67.31 0)
       (effects (font (size 1.27 1.27)) hide)
     )
@@
     )
     (path "/62bde10e-00a3-4c9f-8511-9b691a7797c4"
-      (reference "J2") (unit 1) (value "powerin") (footprint "Connector_Wire:SolderWire-1sqmm_1x02_P5.4mm_D1.4mm_OD2.7mm")
+      (reference "J2") (unit 1) (value "powerin") (footprint "beetleback:beetlepower_in")
     )
     (path "/13b79033-d552-42ca-ba14-db71e8ae705b"

Commit message: tweaks
Parts:
- J1: footprint Connector_PinHeader_2.54mm:PinHeader_1x03_P2.54mm_Vertical -> beetleback:rx_pins
Changed lines of the file:
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@@
     (property "Reference" "J1" (id 0) (at 23.0124 35.56 0))
     (property "Value" "signalin" (id 1) (at 23.0124 38.1 0))
-    (property "Footprint" "Connector_PinHeader_2.54mm:PinHeader_1x03_P2.54mm_Vertical" (id 2) (at 20.32 43.815 0)
+    (property "Footprint" "beetleback:rx_pins" (id 2) (at 20.32 43.815 0)
       (effects (font (size 1.27 1.27)) hide)
     )
@@
     )
     (path "/0e9c9460-869c-49ce-8575-fbed689c08a1"
-      (reference "J1") (unit 1) (value "signalin") (footprint "Connector_PinHeader_2.54mm:PinHeader_1x03_P2.54mm_Vertical")
+      (reference "J1") (unit 1) (value "signalin") (footprint "beetleback:rx_pins")
     )
     (path "/62bde10e-00a3-4c9f-8511-9b691a7797c4"

Commit message: old ideas
Parts:
- U1: LCSC C14075 -> C40382
- U5: value HT75C0-2 -> HT75C0-3; LCSC C95005 -> C259861
Other:
- note added: "HT75C0-3 sot23-5 pins gnd,in,out,nc,nc 12v reg for gate drivers"
- note removed: "HT75C0-2 sot23-5 pins gnd,in,out,nc,nc 12v reg for gate drivers"
Changed lines of the file:
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@@
     (effects (font (size 1.27 1.27)) (justify right bottom))
   )
-  (text "HT75C0-2\nsot23-5 pins gnd,in,out,nc,nc\n12v reg for gate drivers"
+  (text "HT75C0-3\nsot23-5 pins gnd,in,out,nc,nc\n12v reg for gate drivers"
     (at 29.21 111.125 0)
     (effects (font (size 1.27 1.27)) (justify left bottom))
@@
     (in_bom yes) (on_board yes)
     (property "Reference" "U5" (id 0) (at 43.815 114.5348 0))
-    (property "Value" "HT75C0-2" (id 1) (at 43.815 116.8335 0))
+    (property "Value" "HT75C0-3" (id 1) (at 43.815 116.8335 0))
     (property "Footprint" "Package_TO_SOT_SMD:SOT-23-5" (id 2) (at 43.815 115.57 0)
       (effects (font (size 1.27 1.27) italic) hide)
@@
       (effects (font (size 1.27 1.27)) hide)
     )
-    (property "LCSC" "C95005" (id 4) (at 43.815 123.825 0)
+    (property "LCSC" "C259861" (id 4) (at 43.815 123.825 0)
       (effects (font (size 1.27 1.27)) hide)
     )
@@
       (effects (font (size 1.27 1.27)) hide)
     )
-    (property "LCSC" "C14075" (id 4) (at 163.195 60.96 0)
+    (property "LCSC" "C40382" (id 4) (at 163.195 60.96 0)
       (effects (font (size 1.27 1.27)) hide)
     )
@@
     )
     (path "/f7812907-5546-4857-9cc9-d184016c4d46"
-      (reference "U5") (unit 1) (value "HT75C0-2") (footprint "Package_TO_SOT_SMD:SOT-23-5")
-    )
-  )
+      (reference "U5") (unit 1) (value "HT75C0-3") (footprint "Package_TO_SOT_SMD:SOT-23-5")
+    )
+  )
