File: featheresc/featheresc_logic/featheresc_logic.kicad_pcb (KiCad board)
At the start: 2 copper layers, 100 x 39 mm, 9 parts, among them J7 Interconnect 1, J8 Interconnect 2, Q1 2N7002, Q2 AO3401A, U1 ESP32-WROOM-32, U2 XL1509-ADJE1, U3 AMS1117-3.3

Commit message: Featheresc logic
Parts:
- added C1: 100 nF, Capacitor_SMD:C_0603_1608Metric_Pad1.08x0.95mm_HandSolder, F.Cu at (121.0, 69.0)
- added C10: DNP, Capacitor_SMD:C_0603_1608Metric, F.Cu at (155.8, 75.0)
- added C2: 10uF, Capacitor_SMD:C_1206_3216Metric, F.Cu at (104.8, 73.5)
- added C3: 10uF, Capacitor_SMD:C_1206_3216Metric, F.Cu at (117.3, 66.1)
- added C4: 100 nF, Capacitor_SMD:C_0603_1608Metric_Pad1.08x0.95mm_HandSolder, F.Cu at (109.8, 73.0)
- added C5: 4.7uF 50V, Capacitor_SMD:C_1206_3216Metric_Pad1.33x1.80mm_HandSolder, F.Cu at (129.0, 85.5)
- added C6: 4.7uF 50V, Capacitor_SMD:C_1206_3216Metric_Pad1.33x1.80mm_HandSolder, F.Cu at (137.0, 85.5)
- added C7: 4.7uF 50V, Capacitor_SMD:C_1206_3216Metric_Pad1.33x1.80mm_HandSolder, F.Cu at (161.0, 85.5)
- added C8: 4.7uF 50V, Capacitor_SMD:C_1206_3216Metric_Pad1.33x1.80mm_HandSolder, F.Cu at (170.0, 85.5)
- added C9: 10uF 50V, Capacitor_SMD:C_1206_3216Metric, F.Cu at (156.6, 72.1)
- added D1: SS34, Diode_SMD:D_SMA_Handsoldering, F.Cu at (119.5, 62.1)
- added D2: B5819W, Diode_SMD:D_SOD-123, F.Cu at (133.0, 81.5)
- added D3: B5819W, Diode_SMD:D_SOD-123, F.Cu at (141.0, 81.5)
- added D4: B5819W, Diode_SMD:D_SOD-123, F.Cu at (165.0, 82.0)
- added D5: B5819W, Diode_SMD:D_SOD-123, F.Cu at (173.5, 81.5)
- added L1: 68uH, Inductor_SMD:L_10.4x10.4_H4.8, F.Cu at (108.2, 65.8)
- added R1: 1k, Resistor_SMD:R_0603_1608Metric_Pad0.98x0.95mm_HandSolder, F.Cu at (122.3, 65.7)
- added R2: 3.9k, Resistor_SMD:R_0603_1608Metric_Pad0.98x0.95mm_HandSolder, F.Cu at (116.7, 69.0)
- added R3: 1k, Resistor_SMD:R_0603_1608Metric_Pad0.98x0.95mm_HandSolder, F.Cu at (114.1, 73.0)
- added R4: 33k, Resistor_SMD:R_0603_1608Metric_Pad0.98x0.95mm_HandSolder, F.Cu at (121.0, 77.0)
- added R5: 1k, Resistor_SMD:R_0603_1608Metric_Pad0.98x0.95mm_HandSolder, F.Cu at (121.0, 74.5)
- added R6: 33k, Resistor_SMD:R_0603_1608Metric_Pad0.98x0.95mm_HandSolder, F.Cu at (118.5, 71.5)
- added U4: NCP81155MN, Package_DFN_QFN:DFN-8-1EP_3x3mm_P0.5mm_EP1.66x2.38mm, F.Cu at (133.0, 85.6)
- added U5: NCP81155MN, Package_DFN_QFN:DFN-8-1EP_3x3mm_P0.5mm_EP1.66x2.38mm, F.Cu at (140.6, 85.6)
- added U6: NCP81155MN, Package_DFN_QFN:DFN-8-1EP_3x3mm_P0.5mm_EP1.66x2.38mm, F.Cu at (165.0, 85.5)
- added U7: NCP81155MN, Package_DFN_QFN:DFN-8-1EP_3x3mm_P0.5mm_EP1.66x2.38mm, F.Cu at (173.5, 85.5)
- added U8: 78L12G-AB3-R, Package_TO_SOT_SMD:SOT-89-3, F.Cu at (150.7, 73.4)
- moved U1 2.00 mm to (191.0, 78.0)
Connections:
- J7 pad 11: unconnected-(J7-Pad11) -> /PHASE21
- J7 pad 3: unconnected-(J7-Pad3) -> /GATEH11
- J7 pad 4: unconnected-(J7-Pad4) -> /GATEL11
- J7 pad 5: unconnected-(J7-Pad5) -> /PHASE11
- J7 pad 6: unconnected-(J7-Pad6) -> /GATEL21
- J7 pad 7: unconnected-(J7-Pad7) -> /GATEH21
- J8 pad 11: unconnected-(J8-Pad11) -> /PHASE22
- J8 pad 3: unconnected-(J8-Pad3) -> /GATEH12
- J8 pad 4: unconnected-(J8-Pad4) -> /GATEL12
- J8 pad 5: unconnected-(J8-Pad5) -> /PHASE12
- J8 pad 6: unconnected-(J8-Pad6) -> /GATEL22
- J8 pad 7: unconnected-(J8-Pad7) -> /GATEH22
- U1 pad 13: unconnected-(U1-Pad13) -> /MOTORR_1
- U1 pad 16: unconnected-(U1-Pad16) -> /MOTORF_1
- U1 pad 23: unconnected-(U1-Pad23) -> /MOTOREN_1
- U1 pad 27: unconnected-(U1-Pad27) -> /MOTORF_2
- U1 pad 28: unconnected-(U1-Pad28) -> /MOTORR_2
- U1 pad 30: unconnected-(U1-Pad30) -> /MOTOREN_2
- U1 pad 8: unconnected-(U1-Pad8) -> /ISENSE_IN
- U1 pad 9: unconnected-(U1-Pad9) -> /VSENSE_IN

Commit message: Feather esc logic board
Parts:
- removed U3: AMS1117-3.3, Package_TO_SOT_SMD:SOT-223-3_TabPin2
- added C11: DNP, Capacitor_SMD:C_0603_1608Metric_Pad1.08x0.95mm_HandSolder, F.Cu at (139.0, 74.0)
- added D6: Green, LED_SMD:LED_0805_2012Metric_Pad1.15x1.40mm_HandSolder, F.Cu at (197.0, 84.0)
- added D7: Green BEC ON, LED_SMD:LED_0805_2012Metric_Pad1.15x1.40mm_HandSolder, F.Cu at (108.5, 66.0)
- added J1: RC IN 1, Connector_JST:JST_XA_S03B-XASK-1_1x03_P2.50mm_Horizontal, F.Cu at (111.0, 72.5)
- added J2: RC IN 2, Connector_JST:JST_XA_S03B-XASK-1_1x03_P2.50mm_Horizontal, F.Cu at (111.0, 84.5)
- added R10: 1k, Resistor_SMD:R_0603_1608Metric_Pad0.98x0.95mm_HandSolder, F.Cu at (108.5, 68.0)
- added R11: 100k, Resistor_SMD:R_0603_1608Metric_Pad0.98x0.95mm_HandSolder, F.Cu at (139.0, 70.0)
- added R12: 100k, Resistor_SMD:R_0603_1608Metric_Pad0.98x0.95mm_HandSolder, F.Cu at (168.5, 63.0)
- added R13: 1k, Resistor_SMD:R_0603_1608Metric_Pad0.98x0.95mm_HandSolder, F.Cu at (134.0, 91.0)
- added R14: 33k, Resistor_SMD:R_0603_1608Metric_Pad0.98x0.95mm_HandSolder, F.Cu at (139.0, 76.0)
- added R15: 1k, Resistor_SMD:R_0603_1608Metric_Pad0.98x0.95mm_HandSolder, F.Cu at (139.0, 72.0)
- added R7: 1k, Resistor_SMD:R_0603_1608Metric_Pad0.98x0.95mm_HandSolder, F.Cu at (195.0, 84.0)
- added R8: 1k, Resistor_SMD:R_0603_1608Metric_Pad0.98x0.95mm_HandSolder, F.Cu at (168.5, 65.5)
- added R9: 1k, Resistor_SMD:R_0603_1608Metric_Pad0.98x0.95mm_HandSolder, F.Cu at (139.0, 68.0)
- C3: value 10uF -> DNP; footprint Capacitor_SMD:C_1206_3216Metric -> Capacitor_SMD:C_0603_1608Metric_Pad1.08x0.95mm_HandSolder
- R2: value 3.9k -> 3.3k
- U1: value ESP32-WROOM-32 -> RP2040-Zero; footprint RF_Module:ESP32-WROOM-32 -> featheresc_logic:RP2040-Zero
- moved U2 84.3 mm to (191.0, 78.0), turned to -90 degrees
- moved L1 80.8 mm to (189.0, 67.0), turned to 180 degrees
- moved D1 77.9 mm to (197.0, 70.0), turned to -90 degrees
- moved C2 77.3 mm to (182.0, 72.0), turned to -90 degrees
- moved R1 75.3 mm to (196.9, 76.0), turned to 180 degrees
- moved C1 74.7 mm to (195.0, 79.0), turned to -90 degrees
- moved R2 72.6 mm to (189.1, 73.5), turned to 180 degrees
- moved U1 37.8 mm to (153.5, 73.5), turned to 0 degrees
- moved C3 31.8 mm to (137.0, 91.0), turned to -90 degrees
- moved C4 31.6 mm to (140.0, 64.0), turned to -90 degrees
- moved C9 23.1 mm to (151.0, 94.4), turned to 90 degrees
- moved U8 22.1 mm to (155.4, 95.0), turned to 90 degrees
- moved C10 21.2 mm to (149.0, 95.1), turned to 90 degrees
- moved Q1 18.3 mm to (120.0, 67.0), turned to -90 degrees
- moved U4 13.7 mm to (120.0, 90.0), turned to -90 degrees
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Connections:
- net Net-(D1-Pad1) renamed /REGSW
- C3 pad 1: VLOGIC -> /ISENSE_IN
- C4 pad 1: Net-(C4-Pad1) -> VBEC
- J7 pad 8: unconnected-(J7-Pad8) -> GNDSHUNT
- U1 pad 1: GND -> VBEC
- U1 pad 13: /MOTORR_1 -> unconnected-(U1-Pad13)
- U1 pad 14: /BEC_ENABLE -> unconnected-(U1-Pad14)
- U1 pad 15: GND -> /MOTOREN_2
- U1 pad 16: /MOTORF_1 -> /MOTORR_2
- U1 pad 17: unconnected-(U1-Pad17) -> /MOTORF_2
- U1 pad 18: unconnected-(U1-Pad18) -> /BEC_ENABLE
- U1 pad 2: Net-(C4-Pad1) -> GND
- U1 pad 22: unconnected-(U1-Pad22) -> Net-(U1-Pad22)
- U1 pad 23: /MOTOREN_1 -> unconnected-(U1-Pad23)
- U1 pad 4: unconnected-(U1-Pad4) -> Net-(R11-Pad2)
- U1 pad 5: unconnected-(U1-Pad5) -> /VSENSE_IN
- U1 pad 6: unconnected-(U1-Pad6) -> /ISENSE_IN
- U1 pad 7: unconnected-(U1-Pad7) -> /MOTORF_1
- U1 pad 8: /ISENSE_IN -> /MOTORR_1
- U1 pad 9: /VSENSE_IN -> /MOTOREN_1

Commit message: Feather esc logic board
Parts:
- moved D6 4.00 mm to (193.0, 84.0)
- moved R7 4.00 mm to (191.0, 84.0)
- moved C6 3.40 mm to (132.4, 86.0)
- moved C8 3.30 mm to (182.8, 86.0), turned to 0 degrees
- moved C5 3.20 mm to (123.2, 86.0)
- moved C7 2.30 mm to (175.3, 86.1), turned to 0 degrees
- turned D2 to 180 degrees
- turned D3 to 180 degrees
Connections:
- U1 pad 16: /MOTORR_2 -> /MOTORF_2
- U1 pad 17: /MOTORF_2 -> /MOTORR_2
Routing:
- net VBEC: track 0.00 -> 214.8 mm, vias 0 -> 5
- net +12V: track 0.00 -> 101.1 mm, vias 0 -> 2
- net VBAT: track 0.00 -> 96.7 mm, vias 0 -> 2
- net GND: track 0.00 -> 78.1 mm, vias 0 -> 36
- net /RXIN_1: track 0.00 -> 76.8 mm, vias 0 -> 2
- net /BEC_ENABLE: track 0.00 -> 55.9 mm, vias 0 -> 2
- net /RXIN_2: track 0.00 -> 43.2 mm
- net /MOTOREN_1: track 0.00 -> 35.0 mm, vias 0 -> 3
- net /MOTORF_1: track 0.00 -> 31.7 mm, vias 0 -> 2
- net /ISENSE_IN: track 0.00 -> 27.9 mm, vias 0 -> 2
- net /PHASE21: track 0.00 -> 25.7 mm, vias 0 -> 1
- net /MOTORR_2: track 0.00 -> 25.2 mm
- net /VBEC_SWITCHED: track 0.00 -> 24.9 mm
- net /PHASE22: track 0.00 -> 24.1 mm, vias 0 -> 1
- net /MOTOREN_2: track 0.00 -> 21.8 mm, vias 0 -> 3
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- added copper zone on B.Cu, net GND
- added copper zone on F.Cu, net GND
