File: featheresc/featheresc_logic/gatedrivers.kicad_sch (KiCad schematic)
At the start: 0 parts

Commit message: Featheresc logic
Parts:
- added C5, C6: 4.7uF 50V, Capacitor_SMD:C_1206_3216Metric_Pad1.33x1.80mm_HandSolder, symbol Device:C
- added D2, D3: B5819W, Diode_SMD:D_SOD-123, symbol Device:D_Schottky
- added U4, U5: NCP81155MN, Package_DFN_QFN:DFN-8-1EP_3x3mm_P0.5mm_EP1.66x2.38mm, symbol featheresc_logic:NCP81155MN
Connections:
- new net +12V: D2.2 (A), D3.2 (A), U4.4 (VCC), U5.4 (VCC)
- new net BOOST1: C5.1, D2.1 (K), U4.1 (BST)
- new net BOOST2: C6.1, D3.1 (K), U5.1 (BST)
- new net GATEH1: U4.8 (DRVH)
- new net GATEH2: U5.8 (DRVH)
- new net GATEL1: U4.5 (DRVL)
- new net GATEL2: U5.5 (DRVL)
- new net GND: U4.6 (GND), U4.9 (FLAG), U5.6 (GND), U5.9 (FLAG)
- new net MOTORD1: U4.2 (PWM)
- new net MOTORD2: U5.2 (PWM)
- new net MOTOREN: U4.3 (EN), U5.3 (EN)
- new net PHASE1: C5.2, U4.7 (SW)
- new net PHASE2: C6.2, U5.7 (SW)

Commit message: Feather esc logic board
Parts:
- renumbered C5 to C7, C6 to C8, D2 to D4, D3 to D5, U4 to U6, U5 to U7
Changed lines of the file:
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@@
   (paper "A4")
   (junction (at 82.55 113.03) (diameter 0.9144) (color 0 0 0 0))
+  (junction (at 68.58 86.995) (diameter 0.9144) (color 0 0 0 0))
+  (junction (at 68.58 146.685) (diameter 0.9144) (color 0 0 0 0))
+  (junction (at 68.58 113.03) (diameter 0.9144) (color 0 0 0 0))
   (junction (at 68.58 53.34) (diameter 0.9144) (color 0 0 0 0))
   (junction (at 83.82 53.34) (diameter 0.9144) (color 0 0 0 0))
-  (junction (at 68.58 146.685) (diameter 0.9144) (color 0 0 0 0))
-  (junction (at 68.58 86.995) (diameter 0.9144) (color 0 0 0 0))
-  (junction (at 68.58 113.03) (diameter 0.9144) (color 0 0 0 0))
   (wire (pts (xy 68.58 142.24) (xy 68.58 146.685))
     (stroke (width 0) (type solid) (color 0 0 0 0))
@@
   (symbol (lib_id "Device:C") (at 89.535 119.38 0)
     (in_bom yes) (on_board yes)
-    (property "Reference" "C6" (id 0) (at 92.456 118.231 0)
+    (property "Reference" "C8" (id 0) (at 92.456 118.231 0)
       (effects (font (size 1.27 1.27)) (justify left))
     )
@@
   (symbol (lib_id "featheresc_logic:NCP81155MN") (at 68.58 132.08 0)
     (in_bom yes) (on_board yes)
-    (property "Reference" "U5" (id 0) (at 60.0075 121.92 0))
+    (property "Reference" "U7" (id 0) (at 60.0075 121.92 0))
     (property "Value" "NCP81155MN" (id 1) (at 60.0075 119.38 0))
     (property "Footprint" "Package_DFN_QFN:DFN-8-1EP_3x3mm_P0.5mm_EP1.66x2.38mm" (id 2) (at 68.58 132.08 0)
@@
   (symbol (lib_id "power:GND") (at 68.58 88.9 0)
     (in_bom yes) (on_board yes)
-    (property "Reference" "#PWR09" (id 0) (at 68.58 95.25 0)
+    (property "Reference" "#PWR013" (id 0) (at 68.58 95.25 0)
       (effects (font (size 1.27 1.27)) hide)
     )
@@
   (symbol (lib_id "Device:C") (at 89.535 60.96 0)
     (in_bom yes) (on_board yes)
-    (property "Reference" "C5" (id 0) (at 92.4561 59.8106 0)
+    (property "Reference" "C7" (id 0) (at 92.4561 59.8106 0)
       (effects (font (size 1.27 1.27)) (justify left))
     )
@@
   (symbol (lib_id "power:GND") (at 68.58 150.495 0)
     (in_bom yes) (on_board yes)
-    (property "Reference" "#PWR011" (id 0) (at 68.58 156.845 0)
+    (property "Reference" "#PWR015" (id 0) (at 68.58 156.845 0)
       (effects (font (size 1.27 1.27)) hide)
     )
@@
   (symbol (lib_id "power:+12V") (at 68.58 109.22 0)
     (in_bom yes) (on_board yes)
-    (property "Reference" "#PWR010" (id 0) (at 68.58 113.03 0)
+    (property "Reference" "#PWR014" (id 0) (at 68.58 113.03 0)
       (effects (font (size 1.27 1.27)) hide)
     )
@@
   (symbol (lib_id "Device:D_Schottky") (at 72.39 53.34 180)
     (in_bom yes) (on_board yes) (fields_autoplaced)
-    (property "Reference" "D2" (id 0) (at 72.39 48.26 0))
+    (property "Reference" "D4" (id 0) (at 72.39 48.26 0))
     (property "Value" "B5819W" (id 1) (at 72.39 50.8 0))
     (property "Footprint" "Diode_SMD:D_SOD-123" (id 2) (at 72.39 53.34 0)
@@
   (symbol (lib_id "featheresc_logic:NCP81155MN") (at 68.58 73.66 0)
     (in_bom yes) (on_board yes)
-    (property "Reference" "U4" (id 0) (at 60.0075 63.5 0))
+    (property "Reference" "U6" (id 0) (at 60.0075 63.5 0))
     (property "Value" "NCP81155MN" (id 1) (at 60.0075 60.96 0))
     (property "Footprint" "Package_DFN_QFN:DFN-8-1EP_3x3mm_P0.5mm_EP1.66x2.38mm" (id 2) (at 68.58 73.66 0)
@@
   (symbol (lib_id "power:+12V") (at 68.58 45.72 0)
     (in_bom yes) (on_board yes)
-    (property "Reference" "#PWR08" (id 0) (at 68.58 49.53 0)
+    (property "Reference" "#PWR012" (id 0) (at 68.58 49.53 0)
       (effects (font (size 1.27 1.27)) hide)
     )
@@
   (symbol (lib_id "Device:D_Schottky") (at 74.93 113.03 180)
     (in_bom yes) (on_board yes) (fields_autoplaced)
-    (property "Reference" "D3" (id 0) (at 74.93 107.95 0))
+    (property "Reference" "D5" (id 0) (at 74.93 107.95 0))
     (property "Value" "B5819W" (id 1) (at 74.93 110.49 0))
     (property "Footprint" "Diode_SMD:D_SOD-123" (id 2) (at 74.93 113.03 0)
