File: featheresc/featheresc_logic/motordrive.kicad_sch (KiCad schematic)
At the start: 0 parts

Commit message: Featheresc logic
Parts:
- added C10: DNP, Capacitor_SMD:C_0603_1608Metric, symbol Device:C
- added C9: 10uF 50V, Capacitor_SMD:C_1206_3216Metric, symbol Device:C
- added U8: 78L12G-AB3-R, Package_TO_SOT_SMD:SOT-89-3, symbol Regulator_Linear:L78L12_SOT89
Connections:
- new net +12V: C10.1, C9.1, U8.1 (OUT)
- new net GND: C10.2, C9.2, U8.2 (GND)
- new net VBAT: U8.3 (IN)
Other:
- note added: "Linear regulator for gate drivers"
- note added: "Motor Drive common bits"
Changed lines of the file:
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@@
 (kicad_sch (version 20210621) (generator eeschema)
   (paper "A4")
+  (junction (at 69.215 58.42) (diameter 0) (color 0 0 0 0))
+  (junction (at 80.645 69.85) (diameter 0) (color 0 0 0 0))
+  (junction (at 59.69 69.85) (diameter 0) (color 0 0 0 0))
+  (junction (at 80.645 58.42) (diameter 0) (color 0 0 0 0))
+  (junction (at 69.215 69.85) (diameter 0) (color 0 0 0 0))
+  (wire (pts (xy 59.69 69.85) (xy 59.69 75.565))
+    (stroke (width 0) (type solid) (color 0 0 0 0))
+  )
+  (wire (pts (xy 69.215 66.04) (xy 69.215 69.85))
+    (stroke (width 0) (type solid) (color 0 0 0 0))
+  )
+  (wire (pts (xy 59.69 69.85) (xy 69.215 69.85))
+    (stroke (width 0) (type solid) (color 0 0 0 0))
+  )
+  (wire (pts (xy 67.31 58.42) (xy 69.215 58.42))
+    (stroke (width 0) (type solid) (color 0 0 0 0))
+  )
+  (wire (pts (xy 59.69 66.04) (xy 59.69 69.85))
+    (stroke (width 0) (type default) (color 0 0 0 0))
+  )
+  (wire (pts (xy 80.645 58.42) (xy 116.84 58.42))
+    (stroke (width 0) (type solid) (color 0 0 0 0))
+  )
+  (wire (pts (xy 80.645 69.85) (xy 101.6 69.85))
+    (stroke (width 0) (type default) (color 0 0 0 0))
+  )
+  (wire (pts (xy 45.085 58.42) (xy 52.07 58.42))
+    (stroke (width 0) (type solid) (color 0 0 0 0))
+  )
+  (wire (pts (xy 69.215 69.85) (xy 80.645 69.85))
+    (stroke (width 0) (type default) (color 0 0 0 0))
+  )
+  (wire (pts (xy 69.215 58.42) (xy 80.645 58.42))
+    (stroke (width 0) (type default) (color 0 0 0 0))
+  )
+  (wire (pts (xy 80.645 66.04) (xy 80.645 69.85))
+    (stroke (width 0) (type default) (color 0 0 0 0))
+  )
+  (text "Motor Drive common bits" (at 118.745 26.035 0)
+    (effects (font (size 2.5 2.5)) (justify left bottom))
+  )
+  (text "Linear regulator for gate drivers" (at 99.695 55.88 180)
+    (effects (font (size 1.27 1.27)) (justify right bottom))
+  )
+  (global_label "VBAT" (shape input) (at 45.085 58.42 180)
+    (effects (font (size 1.27 1.27)) (justify right))
+    (property "Intersheet References" "${INTERSHEET_REFS}" (id 0) (at 36.7331 58.4994 0)
+      (effects (font (size 1.27 1.27)) (justify right) hide)
+    )
+  )
+  (symbol (lib_id "Regulator_Linear:L78L12_SOT89") (at 59.69 58.42 0) (unit 1)
+    (in_bom yes) (on_board yes)
+    (property "Reference" "U8" (id 0) (at 59.69 52.3048 0))
+    (property "Value" "78L12G-AB3-R " (id 1) (at 59.69 54.603 0))
+    (property "Footprint" "Package_TO_SOT_SMD:SOT-89-3" (id 2) (at 59.69 53.34 0)
+      (effects (font (size 1.27 1.27) italic) hide)
+    )
+    (property "Datasheet" "http://www.st.com/content/ccc/resource/technical/document/datasheet/15/55/e5/aa/23/5b/43/fd/CD00000446.pdf/files/CD00000446.pdf/jcr:content/translations/en.CD00000446.pdf" (id 3) (at 59.69 59.69 0)
+      (effects (font (size 1.27 1.27)) hide)
+    )
+    (property "LCSC" "C75501" (id 4) (at 59.69 58.42 0)
+      (effects (font (size 1.27 1.27)) hide)
+    )
+    (property "Manufacturer" "Unisonic" (id 5) (at 59.69 58.42 0)
+      (effects (font (size 1.27 1.27)) hide)
+    )
+    (pin "1")
+    (pin "2")
+    (pin "3")
+  )
+  (symbol (lib_id "Device:C") (at 69.215 62.23 0) (unit 1)
+    (in_bom yes) (on_board yes)
+    (property "Reference" "C9" (id 0) (at 69.5961 59.8106 0)
+      (effects (font (size 1.27 1.27)) (justify left))
+    )
+    (property "Value" "10uF 50V" (id 1) (at 69.5961 65.2843 0)
+      (effects (font (size 1.27 1.27)) (justify left))
+    )
+    (property "Footprint" "Capacitor_SMD:C_1206_3216Metric" (id 2) (at 70.1802 66.04 0)
+      (effects (font (size 1.27 1.27)) hide)
+    )
+    (property "Datasheet" "~" (id 3) (at 69.215 62.23 0)
+      (effects (font (size 1.27 1.27)) hide)
+    )
+    (property "LCSC" "C13585" (id 4) (at 69.215 62.23 0)
+      (effects (font (size 1.27 1.27)) hide)
+    )
+    (pin "1")
+    (pin "2")
+  )
+  (symbol (lib_id "Device:C") (at 80.645 62.23 0) (unit 1)
+    (in_bom yes) (on_board yes)
+    (property "Reference" "C10" (id 0) (at 81.026 59.811 0)
+      (effects (font (size 1.27 1.27)) (justify left))
+    )
+    (property "Value" "DNP" (id 1) (at 81.0261 65.2843 0)
+      (effects (font (size 1.27 1.27)) (justify left))
+    )
+    (property "Footprint" "Capacitor_SMD:C_0603_1608Metric" (id 2) (at 81.6102 66.04 0)
+      (effects (font (size 1.27 1.27)) hide)
+    )
+    (property "Datasheet" "~" (id 3) (at 80.645 62.23 0)
+      (effects (font (size 1.27 1.27)) hide)
+    )
+    (property "LCSC" "" (id 4) (at 80.645 62.23 0)
+      (effects (font (size 1.27 1.27)) hide)
+    )
+    (pin "1")
+    (pin "2")
+  )
+  (symbol (lib_id "power:GND") (at 59.69 75.565 0) (unit 1)
+    (in_bom yes) (on_board yes)
+    (property "Reference" "#PWR016" (id 0) (at 59.69 81.915 0)
+      (effects (font (size 1.27 1.27)) hide)
+    )
+    (property "Value" "GND" (id 1) (at 59.8043 79.8894 0))
+    (property "Footprint" "" (id 2) (at 59.69 75.565 0)
+      (effects (font (size 1.27 1.27)) hide)
+    )
+    (property "Datasheet" "" (id 3) (at 59.69 75.565 0)
+      (effects (font (size 1.27 1.27)) hide)
+    )
+    (pin "1")
+  )
+  (symbol (lib_id "power:+12V") (at 116.84 58.42 0) (unit 1)
+    (in_bom yes) (on_board yes)
+    (property "Reference" "#PWR017" (id 0) (at 116.84 62.23 0)
+      (effects (font (size 1.27 1.27)) hide)
+    )
+    (property "Value" "+12V" (id 1) (at 117.2083 54.0956 0))
+    (property "Footprint" "" (id 2) (at 116.84 58.42 0)
+      (effects (font (size 1.27 1.27)) hide)
+    )
+    (property "Datasheet" "" (id 3) (at 116.84 58.42 0)
+      (effects (font (size 1.27 1.27)) hide)
+    )
+    (pin "1")
+  )
 )
