File: featheresc/featheresc_logic/sensing.kicad_sch (KiCad schematic)
At the start: 0 parts

Commit message: Feather esc logic board
Parts:
- added C11, C3: DNP, Capacitor_SMD:C_0603_1608Metric_Pad1.08x0.95mm_HandSolder, symbol Device:C
- added R13, R15: 1k, Resistor_SMD:R_0603_1608Metric_Pad0.98x0.95mm_HandSolder, symbol Device:R
- added R14: 33k, Resistor_SMD:R_0603_1608Metric_Pad0.98x0.95mm_HandSolder, symbol Device:R
Connections:
- new net GND: C11.2, C3.2, R15.1
- new net GNDSHUNT: R13.2
- new net ISENSE: C3.1, R13.1
- new net VBAT: R14.2
- new net VSENSE: C11.1, R14.1, R15.2
Other:
- note added: "Current sensing"
- note added: "The RP2040 ADC has a range of 3.3volts because it shares a supply with the MCU, This could be reduced by adding a vref component in to the ADC_DVDD pin but it isn't routed out in the module, so we'd need a bodge wire."
- note added: "Voltage sensing"
Changed lines of the file:
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@@
 (kicad_sch (version 20210621) (generator eeschema)
   (paper "A4")
+  (junction (at 124.46 84.455) (diameter 0) (color 0 0 0 0))
+  (junction (at 113.03 64.77) (diameter 0) (color 0 0 0 0))
+  (junction (at 136.525 84.455) (diameter 0) (color 0 0 0 0))
+  (wire (pts (xy 136.525 84.455) (xy 136.525 86.995))
+    (stroke (width 0) (type default) (color 0 0 0 0))
+  )
+  (wire (pts (xy 106.68 64.77) (xy 113.03 64.77))
+    (stroke (width 0) (type default) (color 0 0 0 0))
+  )
+  (wire (pts (xy 124.46 84.455) (xy 136.525 84.455))
+    (stroke (width 0) (type default) (color 0 0 0 0))
+  )
+  (wire (pts (xy 136.525 84.455) (xy 140.97 84.455))
+    (stroke (width 0) (type default) (color 0 0 0 0))
+  )
+  (wire (pts (xy 108.585 84.455) (xy 124.46 84.455))
+    (stroke (width 0) (type default) (color 0 0 0 0))
+  )
+  (wire (pts (xy 136.525 94.615) (xy 136.525 99.06))
+    (stroke (width 0) (type default) (color 0 0 0 0))
+  )
+  (wire (pts (xy 113.03 64.77) (xy 135.255 64.77))
+    (stroke (width 0) (type default) (color 0 0 0 0))
+  )
+  (wire (pts (xy 124.46 92.075) (xy 124.46 97.155))
+    (stroke (width 0) (type default) (color 0 0 0 0))
+  )
+  (wire (pts (xy 96.52 84.455) (xy 100.965 84.455))
+    (stroke (width 0) (type default) (color 0 0 0 0))
+  )
+  (wire (pts (xy 96.52 64.77) (xy 99.06 64.77))
+    (stroke (width 0) (type default) (color 0 0 0 0))
+  )
+  (text "Current sensing" (at 107.95 57.785 0)
+    (effects (font (size 1.27 1.27)) (justify left bottom))
+  )
+  (text "Voltage sensing" (at 133.35 81.915 0)
+    (effects (font (size 1.27 1.27)) (justify left bottom))
+  )
+  (text "The RP2040 ADC has a range of 3.3volts because it\nshares a supply with the MCU,\n\nThis could be reduced by adding a vref component in\nto the ADC_DVDD pin but it isn't routed out in\nthe module, so we'd need a bodge wire."
+    (at 110.49 50.8 0)
+    (effects (font (size 1.27 1.27)) (justify left bottom))
+  )
+  (global_label "VBAT" (shape input) (at 96.52 84.455 180) (fields_autoplaced)
+    (effects (font (size 1.27 1.27)) (justify right))
+    (property "Intersheet References" "${INTERSHEET_REFS}" (id 0) (at 89.6921 84.5344 0)
+      (effects (font (size 1.27 1.27)) (justify right) hide)
+    )
+  )
+  (global_label "GNDSHUNT" (shape input) (at 96.52 64.77 180) (fields_autoplaced)
+    (effects (font (size 1.27 1.27)) (justify right))
+    (property "Intersheet References" "${INTERSHEET_REFS}" (id 0) (at 84.0679 64.8494 0)
+      (effects (font (size 1.27 1.27)) (justify right) hide)
+    )
+  )
+  (hierarchical_label "ISENSE" (shape input) (at 135.255 64.77 0)
+    (effects (font (size 1.27 1.27)) (justify left))
+  )
+  (hierarchical_label "VSENSE" (shape input) (at 140.97 84.455 0)
+    (effects (font (size 1.27 1.27)) (justify left))
+  )
+  (symbol (lib_id "Device:R") (at 102.87 64.77 270) (unit 1)
+    (in_bom yes) (on_board yes) (fields_autoplaced)
+    (property "Reference" "R13" (id 0) (at 102.87 58.42 90))
+    (property "Value" "1k" (id 1) (at 102.87 60.96 90))
+    (property "Footprint" "Resistor_SMD:R_0603_1608Metric_Pad0.98x0.95mm_HandSolder" (id 2) (at 102.87 62.992 90)
+      (effects (font (size 1.27 1.27)) hide)
+    )
+    (property "Datasheet" "~" (id 3) (at 102.87 64.77 0)
+      (effects (font (size 1.27 1.27)) hide)
+    )
+    (pin "1")
+    (pin "2")
+  )
+  (symbol (lib_id "power:GND") (at 136.525 99.06 0) (unit 1)
+    (in_bom yes) (on_board yes) (fields_autoplaced)
+    (property "Reference" "#PWR024" (id 0) (at 136.525 105.41 0)
+      (effects (font (size 1.27 1.27)) hide)
+    )
+    (property "Value" "GND" (id 1) (at 136.525 103.505 0))
+    (property "Footprint" "" (id 2) (at 136.525 99.06 0)
+      (effects (font (size 1.27 1.27)) hide)
+    )
+    (property "Datasheet" "" (id 3) (at 136.525 99.06 0)
+      (effects (font (size 1.27 1.27)) hide)
+    )
+    (pin "1")
+  )
+  (symbol (lib_id "power:GND") (at 113.03 72.39 0) (unit 1)
+    (in_bom yes) (on_board yes) (fields_autoplaced)
+    (property "Reference" "#PWR022" (id 0) (at 113.03 78.74 0)
+      (effects (font (size 1.27 1.27)) hide)
+    )
+    (property "Value" "GND" (id 1) (at 113.03 76.835 0))
+    (property "Footprint" "" (id 2) (at 113.03 72.39 0)
+      (effects (font (size 1.27 1.27)) hide)
+    )
+    (property "Datasheet" "" (id 3) (at 113.03 72.39 0)
+      (effects (font (size 1.27 1.27)) hide)
+    )
+    (pin "1")
+  )
+  (symbol (lib_id "Device:C") (at 136.525 90.805 0) (unit 1)
+    (in_bom yes) (on_board yes) (fields_autoplaced)
+    (property "Reference" "C11" (id 0) (at 139.7 89.5349 0)
+      (effects (font (size 1.27 1.27)) (justify left))
+    )
+    (property "Value" "DNP" (id 1) (at 139.7 92.0749 0)
+      (effects (font (size 1.27 1.27)) (justify left))
+    )
+    (property "Footprint" "Capacitor_SMD:C_0603_1608Metric_Pad1.08x0.95mm_HandSolder" (id 2) (at 137.4902 94.615 0)
+      (effects (font (size 1.27 1.27)) hide)
+    )
+    (property "Datasheet" "~" (id 3) (at 136.525 90.805 0)
+      (effects (font (size 1.27 1.27)) hide)
+    )
+    (pin "1")
+    (pin "2")
+  )
+  (symbol (lib_id "Device:C") (at 113.03 68.58 0) (unit 1)
+    (in_bom yes) (on_board yes) (fields_autoplaced)
+    (property "Reference" "C3" (id 0) (at 116.84 67.3099 0)
+      (effects (font (size 1.27 1.27)) (justify left))
+    )
+    (property "Value" "DNP" (id 1) (at 116.84 69.8499 0)
+      (effects (font (size 1.27 1.27)) (justify left))
+    )
+    (property "Footprint" "Capacitor_SMD:C_0603_1608Metric_Pad1.08x0.95mm_HandSolder" (id 2) (at 113.9952 72.39 0)
+      (effects (font (size 1.27 1.27)) hide)
+    )
+    (property "Datasheet" "~" (id 3) (at 113.03 68.58 0)
+      (effects (font (size 1.27 1.27)) hide)
+    )
+    (pin "1")
+    (pin "2")
+  )
+  (symbol (lib_id "Device:R") (at 104.775 84.455 270) (unit 1)
+    (in_bom yes) (on_board yes)
+    (property "Reference" "R14" (id 0) (at 103.505 86.995 90))
+    (property "Value" "33k" (id 1) (at 103.505 81.915 90))
+    (property "Footprint" "Resistor_SMD:R_0603_1608Metric_Pad0.98x0.95mm_HandSolder" (id 2) (at 104.775 82.677 90)
+      (effects (font (size 1.27 1.27)) hide)
+    )
+    (property "Datasheet" "~" (id 3) (at 104.775 84.455 0)
+      (effects (font (size 1.27 1.27)) hide)
+    )
+    (pin "1")
+    (pin "2")
+  )
+  (symbol (lib_id "power:GND") (at 124.46 97.155 0) (unit 1)
+    (in_bom yes) (on_board yes) (fields_autoplaced)
+    (property "Reference" "#PWR023" (id 0) (at 124.46 103.505 0)
+      (effects (font (size 1.27 1.27)) hide)
+    )
+    (property "Value" "GND" (id 1) (at 124.46 101.6 0))
+    (property "Footprint" "" (id 2) (at 124.46 97.155 0)
+      (effects (font (size 1.27 1.27)) hide)
+    )
+    (property "Datasheet" "" (id 3) (at 124.46 97.155 0)
+      (effects (font (size 1.27 1.27)) hide)
+    )
+    (pin "1")
+  )
+  (symbol (lib_id "Device:R") (at 124.46 88.265 180) (unit 1)
+    (in_bom yes) (on_board yes) (fields_autoplaced)
+    (property "Reference" "R15" (id 0) (at 126.365 86.9949 0)
+      (effects (font (size 1.27 1.27)) (justify right))
+    )
+    (property "Value" "1k" (id 1) (at 126.365 89.5349 0)
+      (effects (font (size 1.27 1.27)) (justify right))
+    )
+    (property "Footprint" "Resistor_SMD:R_0603_1608Metric_Pad0.98x0.95mm_HandSolder" (id 2) (at 126.238 88.265 90)
+      (effects (font (size 1.27 1.27)) hide)
+    )
+    (property "Datasheet" "~" (id 3) (at 124.46 88.265 0)
+      (effects (font (size 1.27 1.27)) hide)
+    )
+    (pin "1")
+    (pin "2")
+  )
 )
