File: n20_motorback/motorback_panel16/panel16.kicad_pcb (KiCad board)
At the start: 2 copper layers, 124 x 67 mm, 208 parts, among them J1 Servo wire input, J2 Conn_01x01_Male, J3 Conn_01x01_Male, J4 prog_pins, U1 DRV8837DSGR, U2 ATtiny4-TS, U3 AIC1734-33GUTR

Commit message: Panel of 16
Parts:
- removed the C1 at (144.2, 60.9)
- removed the C1 at (144.2, 102.9)
- removed the C1 at (174.2, 102.9)
- removed the C1 at (114.2, 102.9)
- removed the C1 at (114.2, 60.9)
- removed the C1 at (84.2, 74.9)
- removed the C1 at (174.2, 88.9)
- removed the C1 at (174.2, 74.9)
- removed the C1 at (84.2, 88.9)
- removed the C1 at (114.2, 74.9)
- removed the C1 at (174.2, 60.9)
- removed the C1 at (144.2, 88.9)
- removed the C1 at (84.2, 102.9)
- removed the C1 at (114.2, 88.9)
- removed the C1 at (144.2, 74.9)
- removed the C1 at (84.2, 60.9)
- removed the C2 at (86.3, 103.1)
- removed the C2 at (86.3, 89.1)
- removed the C2 at (116.3, 75.1)
- removed the C2 at (146.3, 89.1)
- removed the C2 at (86.3, 75.1)
- removed the C2 at (116.3, 103.1)
- removed the C2 at (146.3, 103.1)
- removed the C2 at (146.3, 61.1)
- removed the C2 at (176.3, 75.1)
- removed the C2 at (146.3, 75.1)
- removed the C2 at (116.3, 61.1)
- removed the C2 at (176.3, 61.1)
- removed the C2 at (176.3, 103.1)
- removed the C2 at (116.3, 89.1)
- removed the C2 at (176.3, 89.1)
- removed the C2 at (86.3, 61.1)
- removed the C3 at (151.0, 79.2)
- removed the C3 at (181.0, 107.2)
- removed the C3 at (181.0, 79.2)
- removed the C3 at (181.0, 65.2)
- removed the C3 at (151.0, 93.2)
- removed the C3 at (91.0, 107.2)
- removed the C3 at (91.0, 93.2)
- removed the C3 at (91.0, 79.2)
- removed the C3 at (151.0, 107.2)
- removed the C3 at (181.0, 93.2)
- removed the C3 at (151.0, 65.2)
- removed the C3 at (121.0, 79.2)
- removed the C3 at (121.0, 93.2)
- removed the C3 at (121.0, 65.2)
- removed the C3 at (121.0, 107.2)
- removed the C3 at (91.0, 65.2)
- removed the U1 at (89.5, 76.0)
- removed the U1 at (149.5, 90.0)
- removed the U1 at (89.5, 104.0)
- removed the U1 at (119.5, 62.0)
- removed the U1 at (149.5, 76.0)
- removed the U1 at (89.5, 62.0)
- removed the U1 at (119.5, 76.0)
- removed the U1 at (119.5, 90.0)
- removed the U1 at (179.5, 62.0)
- removed the U1 at (89.5, 90.0)
- removed the U1 at (179.5, 104.0)
- removed the U1 at (149.5, 62.0)
- removed the U1 at (119.5, 104.0)
- removed the U1 at (179.5, 90.0)
- removed the U1 at (179.5, 76.0)
- removed the U1 at (149.5, 104.0)
- removed the U2 at (93.9, 76.2)
- removed the U2 at (153.9, 62.2)
- removed the U2 at (183.9, 104.2)
- removed the U2 at (153.9, 90.2)
- removed the U2 at (123.9, 76.2)
- removed the U2 at (93.9, 104.2)
- removed the U2 at (153.9, 104.2)
- removed the U2 at (183.9, 90.2)
- removed the U2 at (93.9, 62.2)
- removed the U2 at (183.9, 62.2)
- removed the U2 at (123.9, 104.2)
- removed the U2 at (183.9, 76.2)
- removed the U2 at (93.9, 90.2)
- removed the U2 at (123.9, 62.2)
- removed the U2 at (123.9, 90.2)
- removed the U2 at (153.9, 76.2)
- added C1: 10uF, Capacitor_SMD:C_0603_1608Metric, F.Cu at (112.7, 89.3)
- added C1: 10uF, Capacitor_SMD:C_0603_1608Metric, F.Cu at (172.7, 103.3)
- added C1: 10uF, Capacitor_SMD:C_0603_1608Metric, F.Cu at (172.7, 89.3)
- added C1: 10uF, Capacitor_SMD:C_0603_1608Metric, F.Cu at (142.7, 61.3)
- added C1: 10uF, Capacitor_SMD:C_0603_1608Metric, F.Cu at (172.7, 75.3)
- added C1: 10uF, Capacitor_SMD:C_0603_1608Metric, F.Cu at (82.7, 89.3)
- added C1: 10uF, Capacitor_SMD:C_0603_1608Metric, F.Cu at (112.7, 75.3)
- added C1: 10uF, Capacitor_SMD:C_0603_1608Metric, F.Cu at (142.7, 89.3)
- added C1: 10uF, Capacitor_SMD:C_0603_1608Metric, F.Cu at (82.7, 103.3)
- added C1: 10uF, Capacitor_SMD:C_0603_1608Metric, F.Cu at (82.7, 75.3)
- added C1: 10uF, Capacitor_SMD:C_0603_1608Metric, F.Cu at (142.7, 75.3)
- added C1: 10uF, Capacitor_SMD:C_0603_1608Metric, F.Cu at (82.7, 61.3)
- added C1: 10uF, Capacitor_SMD:C_0603_1608Metric, F.Cu at (112.7, 61.3)
- added C1: 10uF, Capacitor_SMD:C_0603_1608Metric, F.Cu at (172.7, 61.3)
- added C1: 10uF, Capacitor_SMD:C_0603_1608Metric, F.Cu at (112.7, 103.3)
- added C1: 10uF, Capacitor_SMD:C_0603_1608Metric, F.Cu at (142.7, 103.3)
- added C2: 1uF, Capacitor_SMD:C_0603_1608Metric, F.Cu at (115.9, 74.9)
- added C2: 1uF, Capacitor_SMD:C_0603_1608Metric, F.Cu at (85.9, 74.9)
- added C2: 1uF, Capacitor_SMD:C_0603_1608Metric, F.Cu at (175.9, 60.9)
- added C2: 1uF, Capacitor_SMD:C_0603_1608Metric, F.Cu at (175.9, 88.9)
- added C2: 1uF, Capacitor_SMD:C_0603_1608Metric, F.Cu at (115.9, 88.9)
- added C2: 1uF, Capacitor_SMD:C_0603_1608Metric, F.Cu at (175.9, 74.9)
- added C2: 1uF, Capacitor_SMD:C_0603_1608Metric, F.Cu at (85.9, 102.9)
- added C2: 1uF, Capacitor_SMD:C_0603_1608Metric, F.Cu at (145.9, 88.9)
- added C2: 1uF, Capacitor_SMD:C_0603_1608Metric, F.Cu at (85.9, 60.9)
- added C2: 1uF, Capacitor_SMD:C_0603_1608Metric, F.Cu at (175.9, 102.9)
- added C2: 1uF, Capacitor_SMD:C_0603_1608Metric, F.Cu at (145.9, 60.9)
- added C2: 1uF, Capacitor_SMD:C_0603_1608Metric, F.Cu at (85.9, 88.9)
- added C2: 1uF, Capacitor_SMD:C_0603_1608Metric, F.Cu at (115.9, 102.9)
- added C2: 1uF, Capacitor_SMD:C_0603_1608Metric, F.Cu at (145.9, 74.9)
- added C2: 1uF, Capacitor_SMD:C_0603_1608Metric, F.Cu at (145.9, 102.9)
- added C2: 1uF, Capacitor_SMD:C_0603_1608Metric, F.Cu at (115.9, 60.9)
- added C3: 1uF, Capacitor_SMD:C_0603_1608Metric, F.Cu at (180.9, 78.1)
- added C3: 1uF, Capacitor_SMD:C_0603_1608Metric, F.Cu at (90.9, 78.1)
- added C3: 1uF, Capacitor_SMD:C_0603_1608Metric, F.Cu at (90.9, 92.1)
- added C3: 1uF, Capacitor_SMD:C_0603_1608Metric, F.Cu at (120.9, 64.1)
- added C3: 1uF, Capacitor_SMD:C_0603_1608Metric, F.Cu at (120.9, 106.1)
- added C3: 1uF, Capacitor_SMD:C_0603_1608Metric, F.Cu at (180.9, 64.1)
- added C3: 1uF, Capacitor_SMD:C_0603_1608Metric, F.Cu at (90.9, 106.1)
- added C3: 1uF, Capacitor_SMD:C_0603_1608Metric, F.Cu at (120.9, 92.1)
- added C3: 1uF, Capacitor_SMD:C_0603_1608Metric, F.Cu at (180.9, 106.1)
- added C3: 1uF, Capacitor_SMD:C_0603_1608Metric, F.Cu at (150.9, 106.1)
- added C3: 1uF, Capacitor_SMD:C_0603_1608Metric, F.Cu at (120.9, 78.1)
- added C3: 1uF, Capacitor_SMD:C_0603_1608Metric, F.Cu at (150.9, 92.1)
- added C3: 1uF, Capacitor_SMD:C_0603_1608Metric, F.Cu at (150.9, 78.1)
- added C3: 1uF, Capacitor_SMD:C_0603_1608Metric, F.Cu at (150.9, 64.1)
- added C3: 1uF, Capacitor_SMD:C_0603_1608Metric, F.Cu at (90.9, 64.1)
- added C3: 1uF, Capacitor_SMD:C_0603_1608Metric, F.Cu at (180.9, 92.1)
- added U1: BDR6122T, motorback:drv8837_custom, F.Cu at (149.3, 62.1)
- added U1: BDR6122T, motorback:drv8837_custom, F.Cu at (119.3, 62.1)
- added U1: BDR6122T, motorback:drv8837_custom, F.Cu at (119.3, 76.1)
- added U1: BDR6122T, motorback:drv8837_custom, F.Cu at (149.3, 76.1)
- added U1: BDR6122T, motorback:drv8837_custom, F.Cu at (89.3, 90.1)
- added U1: BDR6122T, motorback:drv8837_custom, F.Cu at (179.3, 76.1)
- added U1: BDR6122T, motorback:drv8837_custom, F.Cu at (179.3, 90.1)
- added U1: BDR6122T, motorback:drv8837_custom, F.Cu at (89.3, 104.1)
- added U1: BDR6122T, motorback:drv8837_custom, F.Cu at (119.3, 104.1)
- added U1: BDR6122T, motorback:drv8837_custom, F.Cu at (89.3, 62.1)
- added U1: BDR6122T, motorback:drv8837_custom, F.Cu at (149.3, 104.1)
- added U1: BDR6122T, motorback:drv8837_custom, F.Cu at (119.3, 90.1)
- added U1: BDR6122T, motorback:drv8837_custom, F.Cu at (89.3, 76.1)
- added U1: BDR6122T, motorback:drv8837_custom, F.Cu at (179.3, 62.1)
- added U1: BDR6122T, motorback:drv8837_custom, F.Cu at (149.3, 90.1)
- added U1: BDR6122T, motorback:drv8837_custom, F.Cu at (179.3, 104.1)
- added U2: ATtiny4-MA, Package_DFN_QFN:DFN-8-1EP_2x2mm_P0.5mm_EP0.9x1.5mm, F.Cu at (123.9, 104.2)
- added U2: ATtiny4-MA, Package_DFN_QFN:DFN-8-1EP_2x2mm_P0.5mm_EP0.9x1.5mm, F.Cu at (123.9, 62.2)
- added U2: ATtiny4-MA, Package_DFN_QFN:DFN-8-1EP_2x2mm_P0.5mm_EP0.9x1.5mm, F.Cu at (123.9, 90.2)
- added U2: ATtiny4-MA, Package_DFN_QFN:DFN-8-1EP_2x2mm_P0.5mm_EP0.9x1.5mm, F.Cu at (123.9, 76.2)
- added U2: ATtiny4-MA, Package_DFN_QFN:DFN-8-1EP_2x2mm_P0.5mm_EP0.9x1.5mm, F.Cu at (153.9, 90.2)
- added U2: ATtiny4-MA, Package_DFN_QFN:DFN-8-1EP_2x2mm_P0.5mm_EP0.9x1.5mm, F.Cu at (93.9, 104.2)
- added U2: ATtiny4-MA, Package_DFN_QFN:DFN-8-1EP_2x2mm_P0.5mm_EP0.9x1.5mm, F.Cu at (183.9, 104.2)
- added U2: ATtiny4-MA, Package_DFN_QFN:DFN-8-1EP_2x2mm_P0.5mm_EP0.9x1.5mm, F.Cu at (183.9, 62.2)
- added U2: ATtiny4-MA, Package_DFN_QFN:DFN-8-1EP_2x2mm_P0.5mm_EP0.9x1.5mm, F.Cu at (93.9, 90.2)
- added U2: ATtiny4-MA, Package_DFN_QFN:DFN-8-1EP_2x2mm_P0.5mm_EP0.9x1.5mm, F.Cu at (93.9, 62.2)
- added U2: ATtiny4-MA, Package_DFN_QFN:DFN-8-1EP_2x2mm_P0.5mm_EP0.9x1.5mm, F.Cu at (183.9, 76.2)
- added U2: ATtiny4-MA, Package_DFN_QFN:DFN-8-1EP_2x2mm_P0.5mm_EP0.9x1.5mm, F.Cu at (153.9, 104.2)
- added U2: ATtiny4-MA, Package_DFN_QFN:DFN-8-1EP_2x2mm_P0.5mm_EP0.9x1.5mm, F.Cu at (153.9, 76.2)
- added U2: ATtiny4-MA, Package_DFN_QFN:DFN-8-1EP_2x2mm_P0.5mm_EP0.9x1.5mm, F.Cu at (183.9, 90.2)
- added U2: ATtiny4-MA, Package_DFN_QFN:DFN-8-1EP_2x2mm_P0.5mm_EP0.9x1.5mm, F.Cu at (93.9, 76.2)
- added U2: ATtiny4-MA, Package_DFN_QFN:DFN-8-1EP_2x2mm_P0.5mm_EP0.9x1.5mm, F.Cu at (153.9, 62.2)
Routing:
- net BLINKY: track 182.2 -> 249.2 mm
- net VBAT: track 528.0 -> 477.8 mm
- net /VLOGIC: track 326.8 -> 365.2 mm, vias 16 -> 32
- net /MOTORF: track 141.6 -> 171.3 mm, vias 16 -> 32
- net /MOTORR: track 142.8 -> 171.7 mm
- net GND: track 477.6 -> 451.3 mm
- net /PWMR: track 22.6 -> 34.2 mm
Other:
- board text added: "@markxr 2022"
- board text added: "N20 Motorback Panel16 1.12.2021"
- board text removed: "@markxr 2021"
- board text removed: "N20 Motorback Panel16 16.3.2021"
